File: hardware/ESP32-WROOM.sch (KiCad schematic (older format))
At the start: 5 parts

Commit message: update for DRC,
Parts:
- gave numbers to parts that had none: 5
Connections:
- wire segments 40 -> 43
- no-connect marks 0 -> 12
Changed lines of the file:
@@
 EESchema Schematic File Version 4
-LIBS:AMS1117-cache
+LIBS:RFM95_tryout-cache
 EELAYER 29 0
 EELAYER END
 $Descr A4 11693 8268
 encoding utf-8
-Sheet 2 8
+Sheet 8 8
 Title ""
 Date ""
@@
 $EndDescr
 $Comp
-L taobao-components:ESP-WROOM-32NARROW U?
+L taobao-components:ESP-WROOM-32NARROW U1
 U 1 1 5D0407EC
 P 5950 3700
-F 0 "U?" H 6000 5415 50  0000 C CNN
+F 0 "U1" H 6000 5415 50  0000 C CNN
 F 1 "ESP-WROOM-32NARROW" H 6000 5324 50  0000 C CNN
 F 2 "footprint-lib:ESP-WROOM-32NARROW" H 5950 1350 50  0001 C CNN
@@
 $EndComp
 $Comp
-L power:+3V3 #PWR?
+L power:+3V3 #PWR0101
 U 1 1 5D042BCB
 P 5650 1550
-F 0 "#PWR?" H 5650 1400 50  0001 C CNN
+F 0 "#PWR0101" H 5650 1400 50  0001 C CNN
 F 1 "+3V3" V 5665 1678 50  0000 L CNN
 F 2 "" H 5650 1550 50  0001 C CNN
@@
 $EndComp
 $Comp
-L power:GND #PWR?
+L power:GND #PWR0102
 U 1 1 5D04359B
 P 6400 1550
-F 0 "#PWR?" H 6400 1300 50  0001 C CNN
+F 0 "#PWR0102" H 6400 1300 50  0001 C CNN
 F 1 "GND" V 6405 1422 50  0000 R CNN
 F 2 "" H 6400 1550 50  0001 C CNN
@@
 $EndComp
 $Comp
-L taobao-c:C106,0603 C?
+L taobao-c:C106,0603 C1
 U 1 1 5D043E4F
 P 6000 1550
-F 0 "C?" V 5771 1550 50  0000 C CNN
+F 0 "C1" V 5771 1550 50  0000 C CNN
 F 1 "C106,0603" V 5862 1550 50  0000 C CNN
 F 2 "Capacitor_SMD:C_0603_1608Metric_Pad1.05x0.95mm_HandSolder" H 6000 1550 50  0001 C CNN
@@
 	6100 1550 6400 1550
 $Comp
-L power:+3V3 #PWR?
+L power:+3V3 #PWR0103
 U 1 1 5D044317
 P 5650 1800
-F 0 "#PWR?" H 5650 1650 50  0001 C CNN
+F 0 "#PWR0103" H 5650 1650 50  0001 C CNN
 F 1 "+3V3" V 5665 1928 50  0000 L CNN
 F 2 "" H 5650 1800 50  0001 C CNN
@@
 $EndComp
 $Comp
-L power:GND #PWR?
+L power:GND #PWR0104
 U 1 1 5D044321
 P 6400 1800
-F 0 "#PWR?" H 6400 1550 50  0001 C CNN
+F 0 "#PWR0104" H 6400 1550 50  0001 C CNN
 F 1 "GND" V 6405 1672 50  0000 R CNN
 F 2 "" H 6400 1800 50  0001 C CNN
@@
 	6100 1800 6400 1800
 $Comp
-L taobao-c:C104,0603 C?
+L taobao-c:C104,0603 C2
 U 1 1 5D044EF9
 P 6000 1800
-F 0 "C?" V 5771 1800 50  0000 C CNN
+F 0 "C2" V 5771 1800 50  0000 C CNN
 F 1 "C104,0603" V 5862 1800 50  0000 C CNN
 F 2 "Capacitor_SMD:C_0603_1608Metric_Pad1.05x0.95mm_HandSolder" H 6000 1800 50  0001 C CNN
@@
 $EndComp
 $Comp
-L power:+3V3 #PWR?
+L power:+3V3 #PWR0105
 U 1 1 5D046D95
 P 3550 1750
-F 0 "#PWR?" H 3550 1600 50  0001 C CNN
+F 0 "#PWR0105" H 3550 1600 50  0001 C CNN
 F 1 "+3V3" H 3565 1923 50  0000 C CNN
 F 2 "" H 3550 1750 50  0001 C CNN
@@
 $EndComp
 $Comp
-L taobao-r:R103,0603 R?
+L taobao-r:R103,0603 R1
 U 1 1 5D047495
 P 3050 2050
-F 0 "R?" H 3109 2096 50  0000 L CNN
+F 0 "R1" H 3109 2096 50  0000 L CNN
 F 1 "R103,0603" H 3109 2005 50  0000 L CNN
 F 2 "Resistor_SMD:R_0603_1608Metric_Pad1.05x0.95mm_HandSolder" H 3050 2050 50  0001 C CNN
@@
 RESET
 $Comp
-L taobao-c:C104,0603 C?
+L taobao-c:C104,0603 C3
 U 1 1 5D047E59
 P 3400 2600
-F 0 "C?" H 3492 2646 50  0000 L CNN
+F 0 "C3" H 3492 2646 50  0000 L CNN
 F 1 "C104,0603" H 3492 2555 50  0000 L CNN
 F 2 "Capacitor_SMD:C_0603_1608Metric_Pad1.05x0.95mm_HandSolder" H 3400 2600 50  0001 C CNN
@@
 	3400 2400 3050 2400
 $Comp
-L power:GND #PWR?
+L power:GND #PWR0106
 U 1 1 5D04906C
 P 3400 2800
-F 0 "#PWR?" H 3400 2550 50  0001 C CNN
+F 0 "#PWR0106" H 3400 2550 50  0001 C CNN
 F 1 "GND" H 3405 2627 50  0000 C CNN
 F 2 "" H 3400 2800 50  0001 C CNN
@@
 	3400 2800 3400 2700
 $Comp
-L power:GND #PWR?
+L power:GND #PWR0107
 U 1 1 5D04A372
 P 3900 5850
-F 0 "#PWR?" H 3900 5600 50  0001 C CNN
+F 0 "#PWR0107" H 3900 5600 50  0001 C CNN
 F 1 "GND" H 3905 5677 50  0000 C CNN
 F 2 "" H 3900 5850 50  0001 C CNN
@@
 $EndComp
 Wire Wire Line
-	3900 5850 3900 5200
+	3900 5850 3900 5500
 Wire Wire Line
 	3900 5200 4100 5200
@@
 EndData
 $EndBitmap
+Connection ~ 3900 5300
+Wire Wire Line
+	3900 5300 3900 5200
+Connection ~ 3900 5400
+Connection ~ 3900 5500
+NoConn ~ 7900 3200
+Wire Wire Line
+	3900 5400 3900 5300
+Wire Wire Line
+	3900 5500 3900 5400
+NoConn ~ 7900 3800
+NoConn ~ 7900 5200
+NoConn ~ 7900 5300
+NoConn ~ 7900 5400
+NoConn ~ 7900 5500
+NoConn ~ 4100 3200
+NoConn ~ 4100 3300
+NoConn ~ 4100 3400
+NoConn ~ 4100 3500
+NoConn ~ 4100 3600
+NoConn ~ 4100 3700
 $EndSCHEMATC
