File: hardware/LED_BUTTONS.sch (KiCad schematic (older format))
At the start: 5 parts

Commit message: update for DRC,
Parts:
- gave numbers to parts that had none: 5
Changed lines of the file:
@@
 EESchema Schematic File Version 4
-LIBS:AMS1117-cache
+LIBS:RFM95_tryout-cache
 EELAYER 29 0
 EELAYER END
 $Descr User 8500 5500
 encoding utf-8
-Sheet 8 8
+Sheet 7 8
 Title ""
 Date ""
@@
 IO17
 $Comp
-L taobao-r:R103,0603 R?
+L taobao-r:R103,0603 R7
 U 1 1 5D05DFAE
 P 1650 1750
-F 0 "R?" V 1454 1750 50  0000 C CNN
+F 0 "R7" V 1454 1750 50  0000 C CNN
 F 1 "R103,0603" V 1545 1750 50  0000 C CNN
 F 2 "Resistor_SMD:R_0603_1608Metric_Pad1.05x0.95mm_HandSolder" H 1650 1750 50  0001 C CNN
@@
 $EndComp
 $Comp
-L taobao-led:LED_BLUE,0603 D?
+L taobao-led:LED_BLUE,0603 D2
 U 1 1 5D05E4AF
 P 2000 2050
-F 0 "D?" V 2046 1982 50  0000 R CNN
+F 0 "D2" V 2046 1982 50  0000 R CNN
 F 1 "LED_BLUE,0603" V 1955 1982 50  0000 R CNN
 F 2 "footprint-lib:LED_0603_1608Metric" V 2000 2050 50  0001 C CNN
@@
 $EndComp
 $Comp
-L power:GND #PWR?
+L power:GND #PWR0135
 U 1 1 5D05E907
 P 2000 2400
-F 0 "#PWR?" H 2000 2150 50  0001 C CNN
+F 0 "#PWR0135" H 2000 2150 50  0001 C CNN
 F 1 "GND" H 2005 2227 50  0000 C CNN
 F 2 "" H 2000 2400 50  0001 C CNN
@@
 	2000 2150 2000 2400
 $Comp
-L taobao-button:SW_RESET,2_leg,SMD SW?
+L taobao-button:SW_RESET,2_leg,SMD SW1
 U 1 1 5D05F657
 P 1400 1000
-F 0 "SW?" H 1400 1285 50  0000 C CNN
+F 0 "SW1" H 1400 1285 50  0000 C CNN
 F 1 "SW_RESET,2_leg,SMD" H 1400 1194 50  0000 C CNN
 F 2 "footprint-lib:SW_SPST_CK_RS282G05A3" H 1400 1200 50  0001 C CNN
@@
 $EndComp
 $Comp
-L power:GND #PWR?
+L power:GND #PWR0136
 U 1 1 5D05FC33
 P 1000 1250
-F 0 "#PWR?" H 1000 1000 50  0001 C CNN
+F 0 "#PWR0136" H 1000 1000 50  0001 C CNN
 F 1 "GND" H 1005 1077 50  0000 C CNN
 F 2 "" H 1000 1250 50  0001 C CNN
@@
 	1600 1000 2150 1000
 $Comp
-L power:+3V3 #PWR?
+L power:+3V3 #PWR0137
 U 1 1 5D0602B4
 P 2000 2950
-F 0 "#PWR?" H 2000 2800 50  0001 C CNN
+F 0 "#PWR0137" H 2000 2800 50  0001 C CNN
 F 1 "+3V3" H 2015 3123 50  0000 C CNN
 F 2 "" H 2000 2950 50  0001 C CNN
@@
 $EndComp
 $Comp
-L taobao-r:R103,0603 R?
+L taobao-r:R103,0603 R8
 U 1 1 5D06073D
 P 2000 3300
-F 0 "R?" H 2059 3346 50  0000 L CNN
+F 0 "R8" H 2059 3346 50  0000 L CNN
 F 1 "R103,0603" H 2059 3255 50  0000 L CNN
 F 2 "Resistor_SMD:R_0603_1608Metric_Pad1.05x0.95mm_HandSolder" H 2000 3300 50  0001 C CNN
@@
 $EndComp
 $Comp
-L taobao-button:SW_RESET,2_leg,SMD SW?
+L taobao-button:SW_RESET,2_leg,SMD SW2
 U 1 1 5D060B00
 P 1500 3600
-F 0 "SW?" H 1500 3885 50  0000 C CNN
+F 0 "SW2" H 1500 3885 50  0000 C CNN
 F 1 "SW_RESET,2_leg,SMD" H 1500 3794 50  0000 C CNN
 F 2 "footprint-lib:SW_SPST_CK_RS282G05A3" H 1500 3800 50  0001 C CNN
@@
 $EndComp
 $Comp
-L power:GND #PWR?
+L power:GND #PWR0138
 U 1 1 5D061071
 P 1200 3800
-F 0 "#PWR?" H 1200 3550 50  0001 C CNN
+F 0 "#PWR0138" H 1200 3550 50  0001 C CNN
 F 1 "GND" H 1205 3627 50  0000 C CNN
 F 2 "" H 1200 3800 50  0001 C CNN
