File: hardware/RFM95HW.sch (KiCad schematic (older format))
At the start: 5 parts

Commit message: update for DRC,
Parts:
- gave numbers to parts that had none: 5
Connections:
- no-connect marks 0 -> 3
Changed lines of the file:
@@
 EESchema Schematic File Version 4
-LIBS:AMS1117-cache
+LIBS:RFM95_tryout-cache
 EELAYER 29 0
 EELAYER END
 $Descr User 8500 5500
 encoding utf-8
-Sheet 3 8
+Sheet 2 8
 Title ""
 Date ""
@@
 $EndDescr
 $Comp
-L taobao-components:RFM95 U?
+L taobao-components:RFM95 U2
 U 1 1 5D052587
 P 4100 2800
-F 0 "U?" H 4275 3915 50  0000 C CNN
+F 0 "U2" H 4275 3915 50  0000 C CNN
 F 1 "RFM95" H 4275 3824 50  0000 C CNN
 F 2 "footprint-lib:RFM95" H 4100 1700 50  0001 C CNN
@@
 $EndComp
 $Comp
-L power:+3V3 #PWR?
+L power:+3V3 #PWR0108
 U 1 1 5D052DD7
 P 2700 1550
-F 0 "#PWR?" H 2700 1400 50  0001 C CNN
+F 0 "#PWR0108" H 2700 1400 50  0001 C CNN
 F 1 "+3V3" H 2715 1723 50  0000 C CNN
 F 2 "" H 2700 1550 50  0001 C CNN
@@
 $EndComp
 $Comp
-L taobao-r:R103,0603 R?
+L taobao-r:R103,0603 R2
 U 1 1 5D053316
 P 2700 1750
-F 0 "R?" H 2759 1796 50  0000 L CNN
+F 0 "R2" H 2759 1796 50  0000 L CNN
 F 1 "R103,0603" H 2759 1705 50  0000 L CNN
 F 2 "Resistor_SMD:R_0603_1608Metric_Pad1.05x0.95mm_HandSolder" H 2700 1750 50  0001 C CNN
@@
 Connection ~ 2700 2150
 $Comp
-L power:+3V3 #PWR?
+L power:+3V3 #PWR0109
 U 1 1 5D055779
 P 3000 1900
-F 0 "#PWR?" H 3000 1750 50  0001 C CNN
+F 0 "#PWR0109" H 3000 1750 50  0001 C CNN
 F 1 "+3V3" H 3015 2073 50  0000 C CNN
 F 2 "" H 3000 1900 50  0001 C CNN
@@
 	3000 2050 3000 1900
 $Comp
-L taobao-c:C475,0603 C?
+L taobao-c:C475,0603 C4
 U 1 1 5D055F4D
 P 3000 2400
-F 0 "C?" H 3092 2446 50  0000 L CNN
+F 0 "C4" H 3092 2446 50  0000 L CNN
 F 1 "C475,0603" H 3092 2355 50  0000 L CNN
 F 2 "Capacitor_SMD:C_0603_1608Metric_Pad1.05x0.95mm_HandSolder" H 3000 2400 50  0001 C CNN
@@
 	2700 1850 2700 2150
 $Comp
-L power:GND #PWR?
+L power:GND #PWR0110
 U 1 1 5D059300
 P 3000 3550
-F 0 "#PWR?" H 3000 3300 50  0001 C CNN
+F 0 "#PWR0110" H 3000 3300 50  0001 C CNN
 F 1 "GND" H 3005 3377 50  0000 C CNN
 F 2 "" H 3000 3550 50  0001 C CNN
@@
 	5400 2250 5850 2250
 $Comp
-L my_solder_jumper:SolderJumper_2_Open_round JP?
+L my_solder_jumper:SolderJumper_2_Open_round JP1
 U 1 1 5D05B967
 P 3950 850
-F 0 "JP?" H 3950 1055 50  0000 C CNN
+F 0 "JP1" H 3950 1055 50  0000 C CNN
 F 1 "SolderJumper_2_Open_round" H 3950 964 50  0000 C CNN
 F 2 "Jumper:SolderJumper-2_P1.3mm_Open_RoundedPad1.0x1.5mm" H 3950 850 50  0001 C CNN
@@
 ANT
 $Comp
-L power:GND #PWR?
+L power:GND #PWR0111
 U 1 1 5D05BF78
 P 3450 1200
-F 0 "#PWR?" H 3450 950 50  0001 C CNN
+F 0 "#PWR0111" H 3450 950 50  0001 C CNN
 F 1 "GND" H 3455 1027 50  0000 C CNN
 F 2 "" H 3450 1200 50  0001 C CNN
@@
 $EndComp
 $Comp
-L Connector:Conn_01x02_Female J?
+L Connector:Conn_01x02_Female J1
 U 1 1 5D05CA2F
 P 3050 850
-F 0 "J?" H 2942 1035 50  0000 C CNN
+F 0 "J1" H 2942 1035 50  0000 C CNN
 F 1 "Conn_01x02_Female" H 2942 944 50  0000 C CNN
 F 2 "" H 3050 850 50  0001 C CNN
@@
 EndData
 $EndBitmap
+NoConn ~ 5400 2350
+NoConn ~ 5400 2450
+NoConn ~ 5400 2550
 $EndSCHEMATC

Commit message: update,
Parts:
- J1: value Conn_01x02_Female -> ANT; footprint (none) -> Connector_PinHeader_2.54mm:PinHeader_1x02_P2.54mm_Vertical
- JP1: value SolderJumper_2_Open_round -> ANT_EN
Changed lines of the file:
@@
 EESchema Schematic File Version 4
-LIBS:RFM95_tryout-cache
 EELAYER 29 0
 EELAYER END
@@
 P 3950 850
 F 0 "JP1" H 3950 1055 50  0000 C CNN
-F 1 "SolderJumper_2_Open_round" H 3950 964 50  0000 C CNN
+F 1 "ANT_EN" H 3950 964 50  0000 C CNN
 F 2 "Jumper:SolderJumper-2_P1.3mm_Open_RoundedPad1.0x1.5mm" H 3950 850 50  0001 C CNN
 F 3 "~" H 3950 850 50  0001 C CNN
@@
 P 3050 850
 F 0 "J1" H 2942 1035 50  0000 C CNN
-F 1 "Conn_01x02_Female" H 2942 944 50  0000 C CNN
-F 2 "" H 3050 850 50  0001 C CNN
+F 1 "ANT" H 2942 944 50  0000 C CNN
+F 2 "Connector_PinHeader_2.54mm:PinHeader_1x02_P2.54mm_Vertical" H 3050 850 50  0001 C CNN
 F 3 "~" H 3050 850 50  0001 C CNN
 	1    3050 850
