File: hardware/auto_reset.sch (KiCad schematic (older format))
At the start: 4 parts

Commit message: update for DRC,
Parts:
- gave numbers to parts that had none: 4
Changed lines of the file:
@@
 EESchema Schematic File Version 4
-LIBS:AMS1117-cache
+LIBS:RFM95_tryout-cache
 EELAYER 29 0
 EELAYER END
 $Descr User 8500 5500
 encoding utf-8
-Sheet 4 8
+Sheet 3 8
 Title ""
 Date ""
@@
 $EndDescr
 $Comp
-L taobao-transistor:SS9013_J3 Q?
+L taobao-transistor:SS9013_J3 Q1
 U 1 1 5D061FA8
 P 3100 1550
-F 0 "Q?" H 3291 1596 50  0000 L CNN
+F 0 "Q1" H 3291 1596 50  0000 L CNN
 F 1 "SS9013_J3" H 3291 1505 50  0000 L CNN
 F 2 "footprint-lib:9013,J3,SOT23" H 3300 1475 50  0001 L CIN
@@
 $EndComp
 $Comp
-L taobao-transistor:SS9013_J3 Q?
+L taobao-transistor:SS9013_J3 Q2
 U 1 1 5D062695
 P 3100 2350
-F 0 "Q?" H 3291 2304 50  0000 L CNN
+F 0 "Q2" H 3291 2304 50  0000 L CNN
 F 1 "SS9013_J3" H 3291 2395 50  0000 L CNN
 F 2 "footprint-lib:9013,J3,SOT23" H 3300 2275 50  0001 L CIN
@@
 $EndComp
 $Comp
-L taobao-r:R103,0603 R?
+L taobao-r:R103,0603 R4
 U 1 1 5D062C5A
 P 3900 2350
-F 0 "R?" V 3704 2350 50  0000 C CNN
+F 0 "R4" V 3704 2350 50  0000 C CNN
 F 1 "R103,0603" V 3795 2350 50  0000 C CNN
 F 2 "Resistor_SMD:R_0603_1608Metric_Pad1.05x0.95mm_HandSolder" H 3900 2350 50  0001 C CNN
@@
 $EndComp
 $Comp
-L taobao-r:R103,0603 R?
+L taobao-r:R103,0603 R3
 U 1 1 5D062EF1
 P 3900 1550
-F 0 "R?" V 3704 1550 50  0000 C CNN
+F 0 "R3" V 3704 1550 50  0000 C CNN
 F 1 "R103,0603" V 3795 1550 50  0000 C CNN
 F 2 "Resistor_SMD:R_0603_1608Metric_Pad1.05x0.95mm_HandSolder" H 3900 1550 50  0001 C CNN
