File: hardware/auto_reset.sch (KiCad schematic (older format))
At the start: 4 parts, among them Q1 SS9013_J3, Q2 SS9013_J3

Commit message: update,
Parts:
- removed Q1, Q2: SS9013_J3, footprint-lib:9013,J3,SOT23, symbol taobao-transistor:SS9013_J3
- added Q1, Q2: 2N3904(1AM), footprint-lib:MBT3904_1AM_SOT, symbol taobao-transistor:2N3904(1AM)
Changed lines of the file:
@@
 $EndDescr
-$Comp
-L taobao-transistor:SS9013_J3 Q1
-U 1 1 5D061FA8
-P 3100 1550
-F 0 "Q1" H 3291 1596 50  0000 L CNN
-F 1 "SS9013_J3" H 3291 1505 50  0000 L CNN
-F 2 "footprint-lib:9013,J3,SOT23" H 3300 1475 50  0001 L CIN
-F 3 "https://www.fairchildsemi.com/datasheets/2N/2N3904.pdf" H 3100 1550 50  0001 L CNN
-	1    3100 1550
-	-1   0    0    -1
-$EndComp
-$Comp
-L taobao-transistor:SS9013_J3 Q2
-U 1 1 5D062695
-P 3100 2350
-F 0 "Q2" H 3291 2304 50  0000 L CNN
-F 1 "SS9013_J3" H 3291 2395 50  0000 L CNN
-F 2 "footprint-lib:9013,J3,SOT23" H 3300 2275 50  0001 L CIN
-F 3 "https://www.fairchildsemi.com/datasheets/2N/2N3904.pdf" H 3100 2350 50  0001 L CNN
-	1    3100 2350
-	-1   0    0    1
-$EndComp
 $Comp
 L taobao-r:R103,0603 R4
@@
 EndData
 $EndBitmap
+$Comp
+L taobao-transistor:2N3904(1AM) Q2
+U 1 1 5D06D02A
+P 3100 2350
+F 0 "Q2" H 3300 2300 50  0000 L CNN
+F 1 "2N3904(1AM)" H 3300 2350 50  0000 L CNN
+F 2 "footprint-lib:MBT3904_1AM_SOT" H 3300 2275 50  0001 L CIN
+F 3 "https://assets.nexperia.com/documents/data-sheet/MMBT3904.pdf" H 3100 2350 50  0001 L CNN
+	1    3100 2350
+	-1   0    0    1
+$EndComp
+$Comp
+L taobao-transistor:2N3904(1AM) Q1
+U 1 1 5D06DF19
+P 3100 1550
+F 0 "Q1" H 3300 1600 50  0000 L CNN
+F 1 "2N3904(1AM)" H 3300 1550 50  0000 L CNN
+F 2 "footprint-lib:MBT3904_1AM_SOT" H 3300 1475 50  0001 L CIN
+F 3 "https://assets.nexperia.com/documents/data-sheet/MMBT3904.pdf" H 3100 1550 50  0001 L CNN
+	1    3100 1550
+	-1   0    0    -1
+$EndComp
 $EndSCHEMATC
