File: hardware/io_header.sch (KiCad schematic (older format))
At the start: 5 parts

Commit message: update for DRC,
Parts:
- gave numbers to parts that had none: 5
Connections:
- no-connect marks 0 -> 2
Changed lines of the file:
@@
 EESchema Schematic File Version 4
-LIBS:AMS1117-cache
+LIBS:RFM95_tryout-cache
 EELAYER 29 0
 EELAYER END
 $Descr User 8500 5500
 encoding utf-8
-Sheet 5 8
+Sheet 4 8
 Title ""
 Date ""
@@
 $EndDescr
 $Comp
-L Connector:Conn_01x08_Female J?
+L Connector:Conn_01x08_Female J2
 U 1 1 5D087648
 P 1850 1500
-F 0 "J?" H 1742 875 50  0000 C CNN
+F 0 "J2" H 1742 875 50  0000 C CNN
 F 1 "HEADER1" H 1742 966 50  0000 C CNN
 F 2 "" H 1850 1500 50  0001 C CNN
@@
 $EndComp
 $Comp
-L Connector:Conn_01x10_Female J?
+L Connector:Conn_01x10_Female J3
 U 1 1 5D087E08
 P 3400 1650
-F 0 "J?" H 3292 925 50  0000 C CNN
+F 0 "J3" H 3292 925 50  0000 C CNN
 F 1 "HEADER2" H 3292 1016 50  0000 C CNN
 F 2 "" H 3400 1650 50  0001 C CNN
@@
 $EndComp
 $Comp
-L Connector:Conn_01x04_Female J?
+L Connector:Conn_01x04_Female J5
 U 1 1 5D088C0C
 P 4800 2200
-F 0 "J?" H 4692 1775 50  0000 C CNN
+F 0 "J5" H 4692 1775 50  0000 C CNN
 F 1 "I2C_HEADER" H 4692 1866 50  0000 C CNN
 F 2 "" H 4800 2200 50  0001 C CNN
@@
 $EndComp
 $Comp
-L power:GND #PWR?
+L power:GND #PWR0112
 U 1 1 5D0896F4
 P 5250 2650
-F 0 "#PWR?" H 5250 2400 50  0001 C CNN
+F 0 "#PWR0112" H 5250 2400 50  0001 C CNN
 F 1 "GND" H 5255 2477 50  0000 C CNN
 F 2 "" H 5250 2650 50  0001 C CNN
@@
 	5250 2300 5250 2650
 $Comp
-L power:+3V3 #PWR?
+L power:+3V3 #PWR0113
 U 1 1 5D089C79
 P 5150 1150
-F 0 "#PWR?" H 5150 1000 50  0001 C CNN
+F 0 "#PWR0113" H 5150 1000 50  0001 C CNN
 F 1 "+3V3" H 5165 1323 50  0000 C CNN
 F 2 "" H 5150 1150 50  0001 C CNN
@@
 $EndComp
 $Comp
-L taobao-rpack:RN_473,0603 RN?
+L taobao-rpack:RN_473,0603 RN1
 U 1 1 5D08A1A9
 P 5450 1600
-F 0 "RN?" H 5638 1646 50  0000 L CNN
+F 0 "RN1" H 5638 1646 50  0000 L CNN
 F 1 "RN_473,0603" H 5638 1555 50  0000 L CNN
 F 2 "Resistor_SMD:R_Array_Concave_4x0603" V 5725 1600 50  0001 C CNN
@@
 	5350 2100 5000 2100
 $Comp
-L power:+3V3 #PWR?
+L power:+3V3 #PWR0114
 U 1 1 5D0902E5
 P 5450 2500
-F 0 "#PWR?" H 5450 2350 50  0001 C CNN
+F 0 "#PWR0114" H 5450 2350 50  0001 C CNN
 F 1 "+3V3" H 5465 2673 50  0000 C CNN
 F 2 "" H 5450 2500 50  0001 C CNN
@@
 	3600 2050 4100 2050
 $Comp
-L Connector:Conn_01x01_Female J?
+L Connector:Conn_01x01_Female J4
 U 1 1 5D09C1AA
 P 1850 2150
-F 0 "J?" H 1742 2335 50  0000 C CNN
+F 0 "J4" H 1742 2335 50  0000 C CNN
 F 1 "ANT" H 1742 2244 50  0000 C CNN
 F 2 "" H 1850 2150 50  0001 C CNN
@@
 	2550 2150 2050 2150
 $Comp
-L power:GND #PWR?
+L power:GND #PWR0115
 U 1 1 5D0A3799
 P 2650 900
-F 0 "#PWR?" H 2650 650 50  0001 C CNN
+F 0 "#PWR0115" H 2650 650 50  0001 C CNN
 F 1 "GND" H 2655 727 50  0000 C CNN
 F 2 "" H 2650 900 50  0001 C CNN
@@
 	2050 1100 2650 1100
 $Comp
-L power:+3V3 #PWR?
+L power:+3V3 #PWR0116
 U 1 1 5D0A45C0
 P 2900 1050
-F 0 "#PWR?" H 2900 900 50  0001 C CNN
+F 0 "#PWR0116" H 2900 900 50  0001 C CNN
 F 1 "+3V3" H 2915 1223 50  0000 C CNN
 F 2 "" H 2900 1050 50  0001 C CNN
@@
 	2050 1200 2900 1200
 $Comp
-L power:GND #PWR?
+L power:GND #PWR0117
 U 1 1 5D0A5F37
 P 4400 950
-F 0 "#PWR?" H 4400 700 50  0001 C CNN
+F 0 "#PWR0117" H 4400 700 50  0001 C CNN
 F 1 "GND" H 4405 777 50  0000 C CNN
 F 2 "" H 4400 950 50  0001 C CNN
@@
 EndData
 $EndBitmap
+NoConn ~ 5450 1800
+NoConn ~ 5550 1800
 $EndSCHEMATC

Commit message: update,
Parts:
- J2: footprint (none) -> Connector_PinHeader_2.54mm:PinHeader_1x08_P2.54mm_Vertical
- J3: footprint (none) -> Connector_PinHeader_2.54mm:PinHeader_1x10_P2.54mm_Vertical
- J4: footprint (none) -> Connector_PinHeader_2.54mm:PinHeader_1x01_P2.54mm_Vertical
- J5: footprint (none) -> Connector_PinHeader_2.54mm:PinHeader_1x04_P2.54mm_Vertical
Changed lines of the file:
@@
 EESchema Schematic File Version 4
-LIBS:RFM95_tryout-cache
 EELAYER 29 0
 EELAYER END
@@
 F 0 "J2" H 1742 875 50  0000 C CNN
 F 1 "HEADER1" H 1742 966 50  0000 C CNN
-F 2 "" H 1850 1500 50  0001 C CNN
+F 2 "Connector_PinHeader_2.54mm:PinHeader_1x08_P2.54mm_Vertical" H 1850 1500 50  0001 C CNN
 F 3 "~" H 1850 1500 50  0001 C CNN
 	1    1850 1500
@@
 F 0 "J3" H 3292 925 50  0000 C CNN
 F 1 "HEADER2" H 3292 1016 50  0000 C CNN
-F 2 "" H 3400 1650 50  0001 C CNN
+F 2 "Connector_PinHeader_2.54mm:PinHeader_1x10_P2.54mm_Vertical" H 3400 1650 50  0001 C CNN
 F 3 "~" H 3400 1650 50  0001 C CNN
 	1    3400 1650
@@
 F 0 "J5" H 4692 1775 50  0000 C CNN
 F 1 "I2C_HEADER" H 4692 1866 50  0000 C CNN
-F 2 "" H 4800 2200 50  0001 C CNN
+F 2 "Connector_PinHeader_2.54mm:PinHeader_1x04_P2.54mm_Vertical" H 4800 2200 50  0001 C CNN
 F 3 "~" H 4800 2200 50  0001 C CNN
 	1    4800 2200
@@
 F 0 "J4" H 1742 2335 50  0000 C CNN
 F 1 "ANT" H 1742 2244 50  0000 C CNN
-F 2 "" H 1850 2150 50  0001 C CNN
+F 2 "Connector_PinHeader_2.54mm:PinHeader_1x01_P2.54mm_Vertical" H 1850 2150 50  0001 C CNN
 F 3 "~" H 1850 2150 50  0001 C CNN
 	1    1850 2150
