File: hardware/io_header.sch (KiCad schematic (older format))
At the start: 5 parts, among them J2 HEADER1, J3 HEADER2, J4 ANT, J5 I2C_HEADER

Commit message: update,
Connections:
- net SCL: now also J3.1 (Pin_1), RN1.2 (R2.1); no longer J3.2 (Pin_2), RN1.1 (R1.1)
- net SDA: now also J3.2 (Pin_2), RN1.1 (R1.1); no longer J3.1 (Pin_1), RN1.2 (R2.1)
Changed lines of the file:
@@
 L taobao-rpack:RN_473,0603 RN1
 U 1 1 5D08A1A9
-P 5450 1600
-F 0 "RN1" H 5638 1646 50  0000 L CNN
-F 1 "RN_473,0603" H 5638 1555 50  0000 L CNN
-F 2 "Resistor_SMD:R_Array_Concave_4x0603" V 5725 1600 50  0001 C CNN
-F 3 "~" H 5450 1600 50  0001 C CNN
-	1    5450 1600
-	1    0    0    -1
+P 5350 1600
+F 0 "RN1" H 5538 1646 50  0000 L CNN
+F 1 "RN_473,0603" H 5538 1555 50  0000 L CNN
+F 2 "Resistor_SMD:R_Array_Concave_4x0603" V 5625 1600 50  0001 C CNN
+F 3 "~" H 5350 1600 50  0001 C CNN
+	1    5350 1600
+	-1   0    0    -1
 $EndComp
 Wire Wire Line
@@
 	5250 1250 5350 1250
 Wire Wire Line
-	5250 2000 5250 1800
-Wire Wire Line
-	5000 2000 5250 2000
-Wire Wire Line
-	5350 1800 5350 2100
-Wire Wire Line
-	5350 2100 5000 2100
+	5450 2000 5450 1800
+Wire Wire Line
+	5550 1800 5550 2100
 $Comp
 L power:+3V3 #PWR0114
@@
 Wire Wire Line
 	5450 2200 5000 2200
-Text HLabel 5700 2000 2    50   Input ~ 0
-SCL
 Text HLabel 5700 2100 2    50   Input ~ 0
 SDA
 Wire Wire Line
-	5250 2000 5700 2000
-Connection ~ 5250 2000
-Wire Wire Line
-	5700 2100 5350 2100
-Connection ~ 5350 2100
+	5700 2100 5550 2100
 Text HLabel 2550 1300 2    50   Input ~ 0
 RESET
@@
 Text HLabel 4100 1850 2    50   Input ~ 0
 IO4
+Text HLabel 4100 2050 2    50   Input ~ 0
+SCL
 Text HLabel 4100 1950 2    50   Input ~ 0
-SCL
-Text HLabel 4100 2050 2    50   Input ~ 0
 SDA
 Wire Wire Line
@@
 EndData
 $EndBitmap
-NoConn ~ 5450 1800
-NoConn ~ 5550 1800
+NoConn ~ 5250 1800
+NoConn ~ 5350 1800
+Text HLabel 5700 2000 2    50   Input ~ 0
+SCL
+Connection ~ 5450 2000
+Wire Wire Line
+	5450 2000 5700 2000
+Connection ~ 5550 2100
+Wire Wire Line
+	5000 2000 5450 2000
+Wire Wire Line
+	5000 2100 5550 2100
 $EndSCHEMATC
