File: hardware/power.sch (KiCad schematic (older format))
At the start: 11 parts

Commit message: update for DRC,
Parts:
- gave numbers to parts that had none: 11
Changed lines of the file:
@@
 EESchema Schematic File Version 4
-LIBS:AMS1117-cache
+LIBS:RFM95_tryout-cache
 EELAYER 29 0
 EELAYER END
 $Descr User 8500 5500
 encoding utf-8
-Sheet 7 8
+Sheet 6 8
 Title ""
 Date ""
@@
 AR Path="/5C0BFA48/5C0AD747" Ref="U?"  Part="1"
 AR Path="/5C0AD747" Ref="U?"  Part="1"
-AR Path="/5D03FD1B/5C0AD747" Ref="U?"  Part="1"
-F 0 "U?" H 2950 2250 50  0000 C CNN
+AR Path="/5D03FD1B/5C0AD747" Ref="U5"  Part="1"
+F 0 "U5" H 2950 2250 50  0000 C CNN
 F 1 "AMS1117-3.3" H 2950 2150 50  0000 C CNN
 F 2 "Package_TO_SOT_SMD:SOT-223-3_TabPin2" H 2950 2150 50  0001 C CNN
@@
 AR Path="/5C0BFA48/5C0AD74D" Ref="C?"  Part="1"
 AR Path="/5C0AD74D" Ref="C?"  Part="1"
-AR Path="/5D03FD1B/5C0AD74D" Ref="C?"  Part="1"
-F 0 "C?" H 2159 2196 50  0000 R CNN
+AR Path="/5D03FD1B/5C0AD74D" Ref="C6"  Part="1"
+F 0 "C6" H 2159 2196 50  0000 R CNN
 F 1 "C104,0603" H 2159 2105 50  0000 R CNN
 F 2 "Capacitor_SMD:C_0603_1608Metric_Pad1.05x0.95mm_HandSolder" H 2250 2150 50  0001 C CNN
@@
 AR Path="/5C0BFA48/5C0D4463" Ref="#PWR?"  Part="1"
 AR Path="/5C0D4463" Ref="#PWR?"  Part="1"
-AR Path="/5D03FD1B/5C0D4463" Ref="#PWR?"  Part="1"
-F 0 "#PWR?" H 2950 2300 50  0001 C CNN
+AR Path="/5D03FD1B/5C0D4463" Ref="#PWR0124"  Part="1"
+F 0 "#PWR0124" H 2950 2300 50  0001 C CNN
 F 1 "GND" H 3000 2350 50  0000 C CNN
 F 2 "" H 2950 2550 50  0001 C CNN
@@
 AR Path="/5C0BFA48/5C0D4465" Ref="C?"  Part="1"
 AR Path="/5C0D4465" Ref="C?"  Part="1"
-AR Path="/5D03FD1B/5C0D4465" Ref="C?"  Part="1"
-F 0 "C?" H 3592 2196 50  0000 L CNN
+AR Path="/5D03FD1B/5C0D4465" Ref="C7"  Part="1"
+F 0 "C7" H 3592 2196 50  0000 L CNN
 F 1 "C104,0603" H 3592 2105 50  0000 L CNN
 F 2 "Capacitor_SMD:C_0603_1608Metric_Pad1.05x0.95mm_HandSolder" H 3500 2150 50  0001 C CNN
@@
 AR Path="/5C0BFA48/5C04F461" Ref="C?"  Part="1"
 AR Path="/5C04F461" Ref="C?"  Part="1"
-AR Path="/5D03FD1B/5C04F461" Ref="C?"  Part="1"
-F 0 "C?" H 3788 2196 50  0000 L CNN
+AR Path="/5D03FD1B/5C04F461" Ref="C8"  Part="1"
+F 0 "C8" H 3788 2196 50  0000 L CNN
 F 1 "CP47uf,50V" H 3788 2105 50  0000 L CNN
 F 2 "w_smd_cap:c_elec_6.3x7.7" H 3700 2150 50  0001 C CNN
@@
 $EndComp
 $Comp
-L power:+3V3 #PWR?
+L power:+3V3 #PWR0125
 U 1 1 5C0C0902
 P 3700 1500
-F 0 "#PWR?" H 3700 1350 50  0001 C CNN
+F 0 "#PWR0125" H 3700 1350 50  0001 C CNN
 F 1 "+3V3" H 3750 1700 50  0000 C CNN
 F 2 "" H 3700 1500 50  0001 C CNN
@@
 AR Path="/5C0BFA48/5C0C1058" Ref="R?"  Part="1"
 AR Path="/5C0C1058" Ref="R?"  Part="1"
-AR Path="/5D03FD1B/5C0C1058" Ref="R?"  Part="1"
-F 0 "R?" H 2350 3950 50  0000 L CNN
+AR Path="/5D03FD1B/5C0C1058" Ref="R6"  Part="1"
+F 0 "R6" H 2350 3950 50  0000 L CNN
 F 1 "R102,0603" H 2350 3900 50  0000 L CNN
 F 2 "Resistor_SMD:R_0603_1608Metric_Pad1.05x0.95mm_HandSolder" H 2250 3900 50  0001 C CNN
@@
 AR Path="/5D008604/5C0C105F" Ref="#PWR?"  Part="1"
 AR Path="/5C0C105F" Ref="#PWR?"  Part="1"
-AR Path="/5D03FD1B/5C0C105F" Ref="#PWR?"  Part="1"
-F 0 "#PWR?" H 2250 4000 50  0001 C CNN
+AR Path="/5D03FD1B/5C0C105F" Ref="#PWR0126"  Part="1"
+F 0 "#PWR0126" H 2250 4000 50  0001 C CNN
 F 1 "GND" H 2300 4050 50  0000 C CNN
 F 2 "" H 2250 4250 50  0001 C CNN
@@
 	2250 4000 2250 4250
 $Comp
-L power:+3V3 #PWR?
+L power:+3V3 #PWR0127
 U 1 1 5C0C1334
 P 2250 3150
-F 0 "#PWR?" H 2250 3000 50  0001 C CNN
+F 0 "#PWR0127" H 2250 3000 50  0001 C CNN
 F 1 "+3V3" H 2300 3350 50  0000 C CNN
 F 2 "" H 2250 3150 50  0001 C CNN
@@
 $EndComp
 $Comp
-L taobao-led:LED_GREEN,0603 D?
+L taobao-led:LED_GREEN,0603 D1
 U 1 1 5C0D46AA
 P 2250 3550
-F 0 "D?" V 2300 3450 50  0000 R CNN
+F 0 "D1" V 2300 3450 50  0000 R CNN
 F 1 "LED_GREEN,0603" V 2250 3450 50  0000 R CNN
 F 2 "LED_SMD:LED_0603_1608Metric_Pad1.05x0.95mm_HandSolder" V 2250 3550 50  0001 C CNN
@@
 $EndComp
 $Comp
-L Device:Jumper_NO_Small JP?
+L Device:Jumper_NO_Small JP2
 U 1 1 5C148323
 P 2250 1700
-F 0 "JP?" V 2200 1750 50  0000 L CNN
+F 0 "JP2" V 2200 1750 50  0000 L CNN
 F 1 "IN_EN" V 2250 1750 50  0000 L CNN
 F 2 "" H 2250 1700 50  0001 C CNN
@@
 	2250 1800 2250 1950
 $Comp
-L Device:Jumper_NO_Small JP?
+L Device:Jumper_NO_Small JP3
 U 1 1 5C148F3B
 P 3700 1700
-F 0 "JP?" V 3650 1750 50  0000 L CNN
+F 0 "JP3" V 3650 1750 50  0000 L CNN
 F 1 "OUT_EN" V 3700 1750 50  0000 L CNN
 F 2 "" H 3700 1700 50  0001 C CNN
@@
 AR Path="/5C0BFA48/5C14BD92" Ref="#PWR?"  Part="1"
 AR Path="/5C14BD92" Ref="#PWR?"  Part="1"
-AR Path="/5D03FD1B/5C14BD92" Ref="#PWR?"  Part="1"
-F 0 "#PWR?" H 3600 2300 50  0001 C CNN
+AR Path="/5D03FD1B/5C14BD92" Ref="#PWR0128"  Part="1"
+F 0 "#PWR0128" H 3600 2300 50  0001 C CNN
 F 1 "GND" H 3650 2350 50  0000 C CNN
 F 2 "" H 3600 2550 50  0001 C CNN
@@
 AR Path="/5C0BFA48/5C14C0B1" Ref="#PWR?"  Part="1"
 AR Path="/5C14C0B1" Ref="#PWR?"  Part="1"
-AR Path="/5D03FD1B/5C14C0B1" Ref="#PWR?"  Part="1"
-F 0 "#PWR?" H 2250 2300 50  0001 C CNN
+AR Path="/5D03FD1B/5C14C0B1" Ref="#PWR0129"  Part="1"
+F 0 "#PWR0129" H 2250 2300 50  0001 C CNN
 F 1 "GND" H 2300 2350 50  0000 C CNN
 F 2 "" H 2250 2550 50  0001 C CNN
@@
 	2250 2250 2250 2550
 $Comp
-L power:+5V #PWR?
+L power:+5V #PWR0130
 U 1 1 5C153651
 P 2250 1550
-F 0 "#PWR?" H 2250 1400 50  0001 C CNN
+F 0 "#PWR0130" H 2250 1400 50  0001 C CNN
 F 1 "+5V" H 2300 1750 50  0000 C CNN
 F 2 "" H 2250 1550 50  0001 C CNN
@@
 	3700 1500 3700 1600
 $Comp
-L power:+3V3 #PWR?
+L power:+3V3 #PWR0131
 U 1 1 5D00D601
 P 4600 1500
-F 0 "#PWR?" H 4600 1350 50  0001 C CNN
+F 0 "#PWR0131" H 4600 1350 50  0001 C CNN
 F 1 "+3V3" H 4650 1700 50  0000 C CNN
 F 2 "" H 4600 1500 50  0001 C CNN
@@
 $EndComp
 $Comp
-L Connector:TestPoint TP?
+L Connector:TestPoint TP1
 U 1 1 5D00DAC3
 P 4850 1500
-F 0 "TP?" H 4950 1650 50  0000 L CNN
+F 0 "TP1" H 4950 1650 50  0000 L CNN
 F 1 "TP_3V3" H 4950 1550 50  0000 L CNN
 F 2 "Connector_Pin:Pin_D1.0mm_L10.0mm" H 5050 1500 50  0001 C CNN
@@
 	4850 1600 4850 1500
 $Comp
-L power:+5V #PWR?
+L power:+5V #PWR0132
 U 1 1 5D00E788
 P 4600 1900
-F 0 "#PWR?" H 4600 1750 50  0001 C CNN
+F 0 "#PWR0132" H 4600 1750 50  0001 C CNN
 F 1 "+5V" H 4650 2100 50  0000 C CNN
 F 2 "" H 4600 1900 50  0001 C CNN
@@
 $EndComp
 $Comp
-L Connector:TestPoint TP?
+L Connector:TestPoint TP2
 U 1 1 5D00EAB8
 P 4850 1900
-F 0 "TP?" H 4950 2050 50  0000 L CNN
+F 0 "TP2" H 4950 2050 50  0000 L CNN
 F 1 "TP_5V" H 4950 1950 50  0000 L CNN
 F 2 "Connector_Pin:Pin_D1.0mm_L10.0mm" H 5050 1900 50  0001 C CNN
@@
 	4850 2000 4850 1900
 $Comp
-L power:+3V3 #PWR?
+L power:+3V3 #PWR0133
 U 1 1 5D00F2EE
 P 2950 3150
-F 0 "#PWR?" H 2950 3000 50  0001 C CNN
+F 0 "#PWR0133" H 2950 3000 50  0001 C CNN
 F 1 "+3V3" H 3000 3350 50  0000 C CNN
 F 2 "" H 2950 3150 50  0001 C CNN
@@
 AR Path="/5D008604/5D00F59D" Ref="#PWR?"  Part="1"
 AR Path="/5D00F59D" Ref="#PWR?"  Part="1"
-AR Path="/5D03FD1B/5D00F59D" Ref="#PWR?"  Part="1"
-F 0 "#PWR?" H 2950 3500 50  0001 C CNN
+AR Path="/5D03FD1B/5D00F59D" Ref="#PWR0134"  Part="1"
+F 0 "#PWR0134" H 2950 3500 50  0001 C CNN
 F 1 "GND" H 3000 3550 50  0000 C CNN
 F 2 "" H 2950 3750 50  0001 C CNN
@@
 $EndComp
 $Comp
-L taobao-varistor:VAR_3V3,1206 R?
+L taobao-varistor:VAR_3V3,1206 R5
 U 1 1 5D00FCA8
 P 2950 3400
-F 0 "R?" H 3100 3450 50  0000 L CNN
+F 0 "R5" H 3100 3450 50  0000 L CNN
 F 1 "VAR_3V3,1206" H 3100 3400 50  0000 L CNN
 F 2 "footprint-lib:VAR_1206" H 2950 3400 50  0001 C CNN

Commit message: update,
Parts:
- removed JP2: IN_EN, symbol Device:Jumper_NO_Small
- removed JP3: OUT_EN, symbol Device:Jumper_NO_Small
- added JP2: 5V_EN, Jumper:SolderJumper-2_P1.3mm_Open_RoundedPad1.0x1.5mm, symbol my_solder_jumper:SolderJumper_2_Open_round
- added JP3: 3V3_EN, Jumper:SolderJumper-2_P1.3mm_Open_RoundedPad1.0x1.5mm, symbol my_solder_jumper:SolderJumper_2_Open_round
Connections:
- net +3V3: now also JP3.1 (A)
- net +5V: now also JP2.1 (A)
- net at C7.1, C8.1, U5.2 (VO): now also JP3.2 (B)
- net at C6.1, U5.3 (VI): now also JP2.2 (B)
Changed lines of the file:
@@
 EESchema Schematic File Version 4
-LIBS:RFM95_tryout-cache
 EELAYER 29 0
 EELAYER END
@@
 L power:+3V3 #PWR0125
 U 1 1 5C0C0902
-P 3700 1500
-F 0 "#PWR0125" H 3700 1350 50  0001 C CNN
-F 1 "+3V3" H 3750 1700 50  0000 C CNN
-F 2 "" H 3700 1500 50  0001 C CNN
-F 3 "" H 3700 1500 50  0001 C CNN
-	1    3700 1500
+P 3700 1400
+F 0 "#PWR0125" H 3700 1250 50  0001 C CNN
+F 1 "+3V3" H 3750 1600 50  0000 C CNN
+F 2 "" H 3700 1400 50  0001 C CNN
+F 3 "" H 3700 1400 50  0001 C CNN
+	1    3700 1400
 	1    0    0    -1
 $EndComp
@@
 	0    -1   -1   0
 $EndComp
-$Comp
-L Device:Jumper_NO_Small JP2
-U 1 1 5C148323
-P 2250 1700
-F 0 "JP2" V 2200 1750 50  0000 L CNN
-F 1 "IN_EN" V 2250 1750 50  0000 L CNN
-F 2 "" H 2250 1700 50  0001 C CNN
-F 3 "~" H 2250 1700 50  0001 C CNN
-	1    2250 1700
-	0    1    1    0
-$EndComp
-Wire Wire Line
-	2250 1550 2250 1600
+Wire Wire Line
+	2250 1450 2250 1500
 Wire Wire Line
 	2250 1800 2250 1950
-$Comp
-L Device:Jumper_NO_Small JP3
-U 1 1 5C148F3B
-P 3700 1700
-F 0 "JP3" V 3650 1750 50  0000 L CNN
-F 1 "OUT_EN" V 3700 1750 50  0000 L CNN
-F 2 "" H 3700 1700 50  0001 C CNN
-F 3 "~" H 3700 1700 50  0001 C CNN
-	1    3700 1700
-	0    1    1    0
-$EndComp
 Wire Wire Line
 	3700 1800 3700 1950
@@
 L power:+5V #PWR0130
 U 1 1 5C153651
-P 2250 1550
-F 0 "#PWR0130" H 2250 1400 50  0001 C CNN
-F 1 "+5V" H 2300 1750 50  0000 C CNN
-F 2 "" H 2250 1550 50  0001 C CNN
-F 3 "" H 2250 1550 50  0001 C CNN
-	1    2250 1550
-	1    0    0    -1
-$EndComp
-Wire Wire Line
-	3700 1500 3700 1600
+P 2250 1450
+F 0 "#PWR0130" H 2250 1300 50  0001 C CNN
+F 1 "+5V" H 2300 1650 50  0000 C CNN
+F 2 "" H 2250 1450 50  0001 C CNN
+F 3 "" H 2250 1450 50  0001 C CNN
+	1    2250 1450
+	1    0    0    -1
+$EndComp
+Wire Wire Line
+	3700 1400 3700 1500
 $Comp
 L power:+3V3 #PWR0131
@@
 EndData
 $EndBitmap
+$Comp
+L my_solder_jumper:SolderJumper_2_Open_round JP2
+U 1 1 5D042A4E
+P 2250 1650
+F 0 "JP2" V 2204 1718 50  0000 L CNN
+F 1 "5V_EN" V 2295 1718 50  0000 L CNN
+F 2 "Jumper:SolderJumper-2_P1.3mm_Open_RoundedPad1.0x1.5mm" H 2250 1650 50  0001 C CNN
+F 3 "~" H 2250 1650 50  0001 C CNN
+	1    2250 1650
+	0    1    1    0
+$EndComp
+$Comp
+L my_solder_jumper:SolderJumper_2_Open_round JP3
+U 1 1 5D042FDF
+P 3700 1650
+F 0 "JP3" V 3654 1718 50  0000 L CNN
+F 1 "3V3_EN" V 3745 1718 50  0000 L CNN
+F 2 "Jumper:SolderJumper-2_P1.3mm_Open_RoundedPad1.0x1.5mm" H 3700 1650 50  0001 C CNN
+F 3 "~" H 3700 1650 50  0001 C CNN
+	1    3700 1650
+	0    1    1    0
+$EndComp
 $EndSCHEMATC
