File: hardware/power.sch (KiCad schematic (older format))
At the start: 11 parts, among them U5 AMS1117-3.3

Commit message: update,
Parts:
- removed C8: CP47uf,50V, w_smd_cap:c_elec_6.3x7.7, symbol taobao-cp:CP47uf,50V
- added C8: C106,0805, Capacitor_SMD:C_0805_2012Metric_Pad1.15x1.40mm_HandSolder, symbol taobao-c:C106,0805
- U5: footprint Package_TO_SOT_SMD:SOT-223-3_TabPin2 -> footprint-lib:AMS1117_SOT-223
Connections:
- wire segments 28 -> 29
Other:
- moved on the sheet: C7, JP3, TP1, TP2
Changed lines of the file:
@@
 F 0 "U5" H 2950 2250 50  0000 C CNN
 F 1 "AMS1117-3.3" H 2950 2150 50  0000 C CNN
-F 2 "Package_TO_SOT_SMD:SOT-223-3_TabPin2" H 2950 2150 50  0001 C CNN
+F 2 "footprint-lib:AMS1117_SOT-223" H 2950 2150 50  0001 C CNN
 F 3 "http://www.advanced-monolithic.com/pdf/ds1117.pdf" H 3050 1700 50  0001 C CNN
 	1    2950 1950
@@
 $EndComp
 Wire Wire Line
-	3700 2350 3700 2250
+	4250 2350 4250 2250
 Wire Wire Line
 	2250 1950 2650 1950
@@
 	2250 1950 2250 2050
 Wire Wire Line
-	3250 1950 3500 1950
-Connection ~ 3700 1950
-Wire Wire Line
-	3700 1950 3700 2050
+	4250 1950 4250 2050
 $Comp
 L taobao-c:C104,0603 C?
 U 1 1 5C0D4465
-P 3500 2150
+P 4050 2150
 AR Path="/5C0BBB2B/5C0D4465" Ref="C?"  Part="1"
 AR Path="/5C0BFA48/5C0D4465" Ref="C?"  Part="1"
 AR Path="/5C0D4465" Ref="C?"  Part="1"
 AR Path="/5D03FD1B/5C0D4465" Ref="C7"  Part="1"
-F 0 "C7" H 3592 2196 50  0000 L CNN
-F 1 "C104,0603" H 3592 2105 50  0000 L CNN
-F 2 "Capacitor_SMD:C_0603_1608Metric_Pad1.05x0.95mm_HandSolder" H 3500 2150 50  0001 C CNN
-F 3 "~" H 3500 2150 50  0001 C CNN
-	1    3500 2150
-	1    0    0    -1
-$EndComp
-Wire Wire Line
-	3500 2050 3500 1950
-Connection ~ 3500 1950
-Wire Wire Line
-	3500 1950 3700 1950
-Wire Wire Line
-	3500 2250 3500 2350
-Wire Wire Line
-	3500 2350 3600 2350
-$Comp
-L taobao-cp:CP47uf,50V C?
-U 1 1 5C04F461
-P 3700 2150
-AR Path="/5C0BBB2B/5C04F461" Ref="C?"  Part="1"
-AR Path="/5C0BFA48/5C04F461" Ref="C?"  Part="1"
-AR Path="/5C04F461" Ref="C?"  Part="1"
-AR Path="/5D03FD1B/5C04F461" Ref="C8"  Part="1"
-F 0 "C8" H 3788 2196 50  0000 L CNN
-F 1 "CP47uf,50V" H 3788 2105 50  0000 L CNN
-F 2 "w_smd_cap:c_elec_6.3x7.7" H 3700 2150 50  0001 C CNN
-F 3 "~" H 3700 2150 50  0001 C CNN
-	1    3700 2150
-	1    0    0    -1
-$EndComp
+F 0 "C7" H 3950 2200 50  0000 R CNN
+F 1 "C104,0603" H 3950 2150 50  0000 R CNN
+F 2 "Capacitor_SMD:C_0603_1608Metric_Pad1.05x0.95mm_HandSolder" H 4050 2150 50  0001 C CNN
+F 3 "~" H 4050 2150 50  0001 C CNN
+	1    4050 2150
+	1    0    0    -1
+$EndComp
+Wire Wire Line
+	4050 2050 4050 1950
+Wire Wire Line
+	4050 2250 4050 2350
+Wire Wire Line
+	4050 2350 4150 2350
 $Comp
 L power:+3V3 #PWR0125
 U 1 1 5C0C0902
-P 3700 1400
-F 0 "#PWR0125" H 3700 1250 50  0001 C CNN
-F 1 "+3V3" H 3750 1600 50  0000 C CNN
-F 2 "" H 3700 1400 50  0001 C CNN
-F 3 "" H 3700 1400 50  0001 C CNN
-	1    3700 1400
+P 4350 1400
+F 0 "#PWR0125" H 4350 1250 50  0001 C CNN
+F 1 "+3V3" H 4400 1600 50  0000 C CNN
+F 2 "" H 4350 1400 50  0001 C CNN
+F 3 "" H 4350 1400 50  0001 C CNN
+	1    4350 1400
 	1    0    0    -1
 $EndComp
@@
 	2250 1800 2250 1950
 Wire Wire Line
-	3700 1800 3700 1950
+	4350 1800 4350 1950
 Wire Wire Line
 	2950 2250 2950 2550
@@
 L power:GND #PWR?
 U 1 1 5C14BD92
-P 3600 2550
+P 4150 2550
 AR Path="/5C0BBB2B/5C14BD92" Ref="#PWR?"  Part="1"
 AR Path="/5C0BFA48/5C14BD92" Ref="#PWR?"  Part="1"
 AR Path="/5C14BD92" Ref="#PWR?"  Part="1"
 AR Path="/5D03FD1B/5C14BD92" Ref="#PWR0128"  Part="1"
-F 0 "#PWR0128" H 3600 2300 50  0001 C CNN
-F 1 "GND" H 3650 2350 50  0000 C CNN
-F 2 "" H 3600 2550 50  0001 C CNN
-F 3 "" H 3600 2550 50  0001 C CNN
-	1    3600 2550
-	1    0    0    -1
-$EndComp
-Wire Wire Line
-	3600 2350 3600 2550
-Connection ~ 3600 2350
-Wire Wire Line
-	3600 2350 3700 2350
+F 0 "#PWR0128" H 4150 2300 50  0001 C CNN
+F 1 "GND" H 4200 2350 50  0000 C CNN
+F 2 "" H 4150 2550 50  0001 C CNN
+F 3 "" H 4150 2550 50  0001 C CNN
+	1    4150 2550
+	1    0    0    -1
+$EndComp
+Wire Wire Line
+	4150 2350 4150 2550
+Connection ~ 4150 2350
+Wire Wire Line
+	4150 2350 4250 2350
 $Comp
 L power:GND #PWR?
@@
 $EndComp
 Wire Wire Line
-	3700 1400 3700 1500
-$Comp
-L power:+3V3 #PWR0131
-U 1 1 5D00D601
-P 4600 1500
-F 0 "#PWR0131" H 4600 1350 50  0001 C CNN
-F 1 "+3V3" H 4650 1700 50  0000 C CNN
-F 2 "" H 4600 1500 50  0001 C CNN
-F 3 "" H 4600 1500 50  0001 C CNN
-	1    4600 1500
-	1    0    0    -1
-$EndComp
-$Comp
-L Connector:TestPoint TP1
-U 1 1 5D00DAC3
-P 4850 1500
-F 0 "TP1" H 4950 1650 50  0000 L CNN
-F 1 "TP_3V3" H 4950 1550 50  0000 L CNN
-F 2 "Connector_Pin:Pin_D1.0mm_L10.0mm" H 5050 1500 50  0001 C CNN
-F 3 "~" H 5050 1500 50  0001 C CNN
-	1    4850 1500
-	1    0    0    -1
-$EndComp
-Wire Wire Line
-	4600 1500 4600 1600
-Wire Wire Line
-	4600 1600 4850 1600
-Wire Wire Line
-	4850 1600 4850 1500
-$Comp
-L power:+5V #PWR0132
-U 1 1 5D00E788
-P 4600 1900
-F 0 "#PWR0132" H 4600 1750 50  0001 C CNN
-F 1 "+5V" H 4650 2100 50  0000 C CNN
-F 2 "" H 4600 1900 50  0001 C CNN
-F 3 "" H 4600 1900 50  0001 C CNN
-	1    4600 1900
-	1    0    0    -1
-$EndComp
-$Comp
-L Connector:TestPoint TP2
-U 1 1 5D00EAB8
-P 4850 1900
-F 0 "TP2" H 4950 2050 50  0000 L CNN
-F 1 "TP_5V" H 4950 1950 50  0000 L CNN
-F 2 "Connector_Pin:Pin_D1.0mm_L10.0mm" H 5050 1900 50  0001 C CNN
-F 3 "~" H 5050 1900 50  0001 C CNN
-	1    4850 1900
-	1    0    0    -1
-$EndComp
-Wire Wire Line
-	4600 1900 4600 2000
-Wire Wire Line
-	4600 2000 4850 2000
-Wire Wire Line
-	4850 2000 4850 1900
+	4350 1400 4350 1500
+Wire Wire Line
+	5600 2000 5850 2000
 $Comp
 L power:+3V3 #PWR0133
@@
 L my_solder_jumper:SolderJumper_2_Open_round JP3
 U 1 1 5D042FDF
-P 3700 1650
-F 0 "JP3" V 3654 1718 50  0000 L CNN
-F 1 "3V3_EN" V 3745 1718 50  0000 L CNN
-F 2 "Jumper:SolderJumper-2_P1.3mm_Open_RoundedPad1.0x1.5mm" H 3700 1650 50  0001 C CNN
-F 3 "~" H 3700 1650 50  0001 C CNN
-	1    3700 1650
+P 4350 1650
+F 0 "JP3" V 4304 1718 50  0000 L CNN
+F 1 "3V3_EN" V 4395 1718 50  0000 L CNN
+F 2 "Jumper:SolderJumper-2_P1.3mm_Open_RoundedPad1.0x1.5mm" H 4350 1650 50  0001 C CNN
+F 3 "~" H 4350 1650 50  0001 C CNN
+	1    4350 1650
 	0    1    1    0
 $EndComp
+$Comp
+L taobao-c:C106,0805 C8
+U 1 1 5D0724D3
+P 4250 2150
+F 0 "C8" H 4350 2200 50  0000 L CNN
+F 1 "C106,0805" H 4350 2150 50  0000 L CNN
+F 2 "Capacitor_SMD:C_0805_2012Metric_Pad1.15x1.40mm_HandSolder" H 4250 2150 50  0001 C CNN
+F 3 "~" H 4250 2150 50  0001 C CNN
+	1    4250 2150
+	1    0    0    -1
+$EndComp
+Wire Wire Line
+	3250 1950 4050 1950
+Connection ~ 4050 1950
+Wire Wire Line
+	4050 1950 4250 1950
+Connection ~ 4250 1950
+Wire Wire Line
+	4250 1950 4350 1950
+Wire Wire Line
+	5850 2000 5850 1900
+Wire Wire Line
+	5600 1900 5600 2000
+$Comp
+L Connector:TestPoint TP2
+U 1 1 5D00EAB8
+P 5850 1900
+F 0 "TP2" H 5950 2050 50  0000 L CNN
+F 1 "TP_5V" H 5950 1950 50  0000 L CNN
+F 2 "Connector_Pin:Pin_D1.0mm_L10.0mm" H 6050 1900 50  0001 C CNN
+F 3 "~" H 6050 1900 50  0001 C CNN
+	1    5850 1900
+	1    0    0    -1
+$EndComp
+$Comp
+L power:+5V #PWR0132
+U 1 1 5D00E788
+P 5600 1900
+F 0 "#PWR0132" H 5600 1750 50  0001 C CNN
+F 1 "+5V" H 5650 2100 50  0000 C CNN
+F 2 "" H 5600 1900 50  0001 C CNN
+F 3 "" H 5600 1900 50  0001 C CNN
+	1    5600 1900
+	1    0    0    -1
+$EndComp
+Wire Wire Line
+	5850 1600 5850 1500
+Wire Wire Line
+	5600 1600 5850 1600
+Wire Wire Line
+	5600 1500 5600 1600
+$Comp
+L Connector:TestPoint TP1
+U 1 1 5D00DAC3
+P 5850 1500
+F 0 "TP1" H 5950 1650 50  0000 L CNN
+F 1 "TP_3V3" H 5950 1550 50  0000 L CNN
+F 2 "Connector_Pin:Pin_D1.0mm_L10.0mm" H 6050 1500 50  0001 C CNN
+F 3 "~" H 6050 1500 50  0001 C CNN
+	1    5850 1500
+	1    0    0    -1
+$EndComp
+$Comp
+L power:+3V3 #PWR0131
+U 1 1 5D00D601
+P 5600 1500
+F 0 "#PWR0131" H 5600 1350 50  0001 C CNN
+F 1 "+3V3" H 5650 1700 50  0000 C CNN
+F 2 "" H 5600 1500 50  0001 C CNN
+F 3 "" H 5600 1500 50  0001 C CNN
+	1    5600 1500
+	1    0    0    -1
+$EndComp
 $EndSCHEMATC
