File: hardware/usb_to_serial.sch (KiCad schematic (older format))
At the start: 3 parts

Commit message: update for DRC,
Parts:
- gave numbers to parts that had none: 3
Connections:
- net labels added: +5V
- net labels removed: Vusb
- wire segments 32 -> 34
- no-connect marks 0 -> 6
Changed lines of the file:
@@
 EESchema Schematic File Version 4
-LIBS:AMS1117-cache
+LIBS:RFM95_tryout-cache
 EELAYER 29 0
 EELAYER END
 $Descr User 8500 5500
 encoding utf-8
-Sheet 6 8
+Sheet 5 8
 Title ""
 Date ""
@@
 $EndDescr
 $Comp
-L taobao-components:CH340C U?
+L taobao-components:CH340C U4
 U 1 1 5D069003
 P 4300 2000
-F 0 "U?" H 4275 2865 50  0000 C CNN
+F 0 "U4" H 4275 2865 50  0000 C CNN
 F 1 "CH340C" H 4275 2774 50  0000 C CNN
 F 2 "footprint-lib:CH340C" H 4300 550 50  0001 C CNN
@@
 $EndComp
 $Comp
-L taobao-components:USB_Micro U?
+L taobao-components:USB_Micro U3
 U 1 1 5D0698D1
 P 1550 1900
-F 0 "U?" H 1550 2365 50  0000 C CNN
+F 0 "U3" H 1550 2365 50  0000 C CNN
 F 1 "USB_Micro" H 1550 2274 50  0000 C CNN
 F 2 "footprint-lib:USB_Micro-B_Molex-105017-0001" H 1550 1400 50  0001 C CNN
@@
 	2700 1900 3250 1900
 $Comp
-L power:GND #PWR?
+L power:GND #PWR0118
 U 1 1 5D06B994
 P 1000 2350
-F 0 "#PWR?" H 1000 2100 50  0001 C CNN
+F 0 "#PWR0118" H 1000 2100 50  0001 C CNN
 F 1 "GND" H 1005 2177 50  0000 C CNN
 F 2 "" H 1000 2350 50  0001 C CNN
@@
 Connection ~ 1000 2000
 Wire Wire Line
-	1000 2000 1000 1700
+	1000 2000 1000 1800
 Wire Wire Line
 	1150 2100 1000 2100
@@
 Connection ~ 1000 2300
 Wire Wire Line
-	1000 2300 1000 2000
-$Comp
-L my_power:Vusb #PWR?
-U 1 1 5D06C7FE
-P 2150 1350
-F 0 "#PWR?" H 2150 1200 50  0001 C CNN
-F 1 "Vusb" H 2165 1523 50  0000 C CNN
-F 2 "" H 2150 1350 50  0001 C CNN
-F 3 "" H 2150 1350 50  0001 C CNN
-	1    2150 1350
-	1    0    0    -1
-$EndComp
+	1000 2300 1000 2100
 Wire Wire Line
 	2150 1350 2150 1700
@@
 	2150 1700 1950 1700
 $Comp
-L power:+3V3 #PWR?
+L power:+3V3 #PWR0120
 U 1 1 5D06CF89
 P 2950 1250
-F 0 "#PWR?" H 2950 1100 50  0001 C CNN
+F 0 "#PWR0120" H 2950 1100 50  0001 C CNN
 F 1 "+3V3" H 2965 1423 50  0000 C CNN
 F 2 "" H 2950 1250 50  0001 C CNN
@@
 	2950 1500 2950 1600
 $Comp
-L power:GND #PWR?
+L power:GND #PWR0121
 U 1 1 5D06E197
 P 3200 2750
-F 0 "#PWR?" H 3200 2500 50  0001 C CNN
+F 0 "#PWR0121" H 3200 2500 50  0001 C CNN
 F 1 "GND" H 3205 2577 50  0000 C CNN
 F 2 "" H 3200 2750 50  0001 C CNN
@@
 	5300 1800 5850 1800
 $Comp
-L power:+3V3 #PWR?
+L power:+3V3 #PWR0122
 U 1 1 5D06FCFA
 P 3800 3150
-F 0 "#PWR?" H 3800 3000 50  0001 C CNN
+F 0 "#PWR0122" H 3800 3000 50  0001 C CNN
 F 1 "+3V3" V 3815 3278 50  0000 L CNN
 F 2 "" H 3800 3150 50  0001 C CNN
@@
 $EndComp
 $Comp
-L taobao-c:C104,0603 C?
+L taobao-c:C104,0603 C5
 U 1 1 5D07050C
 P 4300 3150
-F 0 "C?" V 4071 3150 50  0000 C CNN
+F 0 "C5" V 4071 3150 50  0000 C CNN
 F 1 "C104,0603" V 4162 3150 50  0000 C CNN
 F 2 "Capacitor_SMD:C_0603_1608Metric_Pad1.05x0.95mm_HandSolder" H 4300 3150 50  0001 C CNN
@@
 $EndComp
 $Comp
-L power:GND #PWR?
+L power:GND #PWR0123
 U 1 1 5D0707B8
 P 4800 3150
-F 0 "#PWR?" H 4800 2900 50  0001 C CNN
+F 0 "#PWR0123" H 4800 2900 50  0001 C CNN
 F 1 "GND" V 4805 3022 50  0000 R CNN
 F 2 "" H 4800 3150 50  0001 C CNN
@@
 EndData
 $EndBitmap
+NoConn ~ 1950 2000
+Connection ~ 1000 1800
+Wire Wire Line
+	1000 1800 1000 1700
+Connection ~ 1000 2100
+Wire Wire Line
+	1000 2100 1000 2000
+NoConn ~ 5300 1900
+NoConn ~ 5300 2000
+NoConn ~ 5300 2100
+NoConn ~ 5300 2200
+NoConn ~ 3250 1700
+$Comp
+L power:+5V #PWR?
+U 1 1 5D073A31
+P 2150 1350
+F 0 "#PWR?" H 2150 1200 50  0001 C CNN
+F 1 "+5V" H 2165 1523 50  0000 C CNN
+F 2 "" H 2150 1350 50  0001 C CNN
+F 3 "" H 2150 1350 50  0001 C CNN
+	1    2150 1350
+	1    0    0    -1
+$EndComp
 $EndSCHEMATC
