File: hardware/ESP32-WROOM_tryout.kicad_pcb (KiCad board)
At the start: 2 copper layers, 100 x 100 mm, 38 parts, among them J1 ANT, J2 HEADER1, J3 HEADER2, J4 ANT, J5 I2C_HEADER, Q1 SS9013_J3, Q2 SS9013_J3, SW1 SW_RESET,2_leg,SMD, SW2 SW_RESET,2_leg,SMD, U1 ESP-WROOM-32NARROW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

Commit message: update,
Parts:
- moved J2 5.00 mm to (105.0, 46.0)
Changed lines of the file:
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@@
   )
   (module Connector_PinHeader_2.54mm:PinHeader_1x08_P2.54mm_Vertical (layer F.Cu)
-    (at 110 46 180)
+    (at 105 46 180)
     (descr "Through hole straight pin header, 1x08, 2.54mm pitch, single row")
     (tags "Through hole pin header THT 1x08 2.54mm single row")

Commit message: update,
Routing:
- net GND: track 0.00 -> 310.4 mm, vias 0 -> 1
- net +3V3: track 0.00 -> 289.3 mm
- net /SCK: track 0.00 -> 102.7 mm
- net /RESET: track 0.00 -> 94.0 mm, vias 0 -> 2
- net +5V: track 0.00 -> 92.0 mm, vias 0 -> 2
- net /MOSI: track 0.00 -> 91.5 mm
- net /SCL: track 0.00 -> 76.3 mm, vias 0 -> 1
- net /SDA: track 0.00 -> 76.2 mm
- net /MISO: track 0.00 -> 72.7 mm, vias 0 -> 1
- net /IO27: track 0.00 -> 66.2 mm, vias 0 -> 1
- net /IO25: track 0.00 -> 63.8 mm, vias 0 -> 1
- net /0: track 0.00 -> 57.0 mm, vias 0 -> 2
- net /RXI: track 0.00 -> 48.9 mm, vias 0 -> 2
- net /TXO: track 0.00 -> 48.8 mm
- net /IO23: track 0.00 -> 38.3 mm, vias 0 -> 1
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
Commit message: update,
Parts:
- C1, C2, C3, C4, C5, JP1, R1, R2, R8, RN1: moved to B.Cu
- C8: value CP47uf,50V -> C106,0805; footprint w_smd_cap:c_elec_6.3x7.7 -> Capacitor_SMD:C_0805_2012Metric_Pad1.15x1.40mm_HandSolder
- Q1, Q2: value SS9013_J3 -> 2N3904(1AM); footprint footprint-lib:9013,J3,SOT23 -> footprint-lib:MBT3904_1AM_SOT
- U5: footprint Package_TO_SOT_SMD:SOT-223-3_TabPin2 -> footprint-lib:AMS1117_SOT-223
- moved SW2 53.9 mm to (96.2, 50.1), turned to 90 degrees
- moved TP2 52.3 mm to (26.7, 25.4)
- moved TP1 51.9 mm to (44.5, 22.4)
- moved C5 51.5 mm to (54.8, 27.0), turned to 0 degrees
- moved R8 50.2 mm to (96.2, 50.1), turned to 90 degrees
- moved J2 42.3 mm to (64.3, 57.5)
- moved R4 41.7 mm to (60.7, 31.5)
- moved U4 40.4 mm to (54.7, 31.5)
- moved U3 40.3 mm to (54.7, 22.5)
- moved C8 39.5 mm to (42.9, 26.8), turned to 270 degrees
- moved R3 38.4 mm to (60.7, 35.5)
- moved R6 36.8 mm to (48.6, 25.8), turned to 180 degrees
- moved D1 35.4 mm to (48.6, 27.6), turned to 180 degrees
- moved RN1 33.4 mm to (93.8, 36.8)
- moved R5 32.9 mm to (45.4, 26.8), turned to 270 degrees
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Connections:
- J3 pad 1: /SDA -> /SCL
- J3 pad 2: /SCL -> /SDA
- RN1 pad 1: /SCL -> /SDA
- RN1 pad 2: /SDA -> /SCL
Routing:
- net +3V3: track 289.3 -> 164.0 mm, vias 0 -> 13
- net /RESET: track 94.0 -> 30.1 mm
- net /SCK: track 102.7 -> 40.8 mm, vias 0 -> 3
- net /IO27: track 66.2 -> 12.7 mm
- net /MOSI: track 91.5 -> 40.2 mm, vias 0 -> 3
- net /IO25: track 63.8 -> 14.4 mm
- net /SDA: track 76.2 -> 27.5 mm, vias 0 -> 1
- net +5V: track 92.0 -> 46.2 mm
- net /SCL: track 76.3 -> 34.7 mm
- net GND: track 310.4 -> 268.8 mm, vias 1 -> 10
- net /MISO: track 72.7 -> 34.1 mm, vias 1 -> 2
- net /RFM95HW/RFM_RST: track 30.4 -> 3.99 mm, vias 0 -> 1
- net /IO23: track 38.3 -> 13.8 mm, vias 1 -> 0
- net /IO19: track 37.6 -> 13.2 mm
- net /IO18: track 36.4 -> 12.7 mm
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Other:
- net class 800mA added: clearance 0.2, trace_width 0.3, via_dia 0.8, via_drill 0.4
- net class GND added: clearance 0.2, trace_width 1.25, via_dia 0.8, via_drill 0.4

Commit message: update,
Parts:
- added C9: C104,0805, Capacitor_SMD:C_0805_2012Metric_Pad1.15x1.40mm_HandSolder, F.Cu at (31.4, 32.4)
- added J6: SHT3x_HEADER, Connector_PinHeader_1.27mm:PinHeader_1x06_P1.27mm_Vertical, F.Cu at (22.5, 30.6)
- added JP4: SolderJumper_2_Open_round, Jumper:SolderJumper-2_P1.3mm_Open_RoundedPad1.0x1.5mm, F.Cu at (33.3, 35.7)
- added JP5: J_ADDR, Jumper:SolderJumper-2_P1.3mm_Open_RoundedPad1.0x1.5mm, F.Cu at (27.7, 32.1)
- added RN2: RN_472,0603, Resistor_SMD:R_Array_Concave_4x0603, B.Cu at (27.7, 35.2)
- added U6: SHT3x-DIS, footprint-lib:SHT3x-DIS, F.Cu at (27.8, 35.2)
Routing:
- net +3V3: track 164.0 -> 201.1 mm, vias 13 -> 16
- net GND: track 268.8 -> 281.6 mm, vias 10 -> 11
- net /SHT3X/NRST: track 0.00 -> 12.4 mm, vias 0 -> 2
- net /SCL: track 34.7 -> 43.3 mm, vias 1 -> 2
- net /SHT3X/ADDR: track 0.00 -> 7.46 mm, vias 0 -> 1
- net /SDA: track 27.5 -> 33.5 mm, vias 1 -> 2
- net Net-(JP4-Pad2): track 0.00 -> 4.96 mm, vias 0 -> 1
- net /SHT3X/ALERT: track 0.00 -> 4.25 mm

Commit message: update,
Parts:
- moved J6 92.9 mm to (112.0, 55.5), turned to 270 degrees
- moved JP5 87.6 mm to (110.5, 60.7), turned to 270 degrees
- moved C9 85.1 mm to (110.2, 64.4), turned to 270 degrees
- moved RN2 83.7 mm to (107.4, 60.7), turned to 270 degrees
- moved U6 83.6 mm to (107.4, 60.8), turned to 270 degrees
- moved JP4 79.8 mm to (106.9, 66.3), turned to 0 degrees
Routing:
- net GND: track 281.6 -> 298.8 mm
- net +3V3: track 201.1 -> 211.7 mm
- net /SDA: track 33.5 -> 43.5 mm
- net /SCL: track 43.3 -> 50.1 mm

Commit message: update,
Parts:
- added H1: MOUNT_M2.5, footprint-lib:MountingHole_2.7mm_M2.5,rpi_like, F.Cu at (25.0, 25.0)
- added H2: MOUNT_M2.5, footprint-lib:MountingHole_2.7mm_M2.5,rpi_like, F.Cu at (25.0, 115.0)
- added H3: MOUNT_M2.5, footprint-lib:MountingHole_2.7mm_M2.5,rpi_like, F.Cu at (115.0, 115.0)
- added H4: MOUNT_M2.5, footprint-lib:MountingHole_2.7mm_M2.5,rpi_like, F.Cu at (115.0, 25.0)
- moved TP2 8.58 mm to (29.5, 33.5)
Routing:
- net +3V3: track 211.7 -> 198.5 mm
- net +5V: track 46.4 -> 51.3 mm
- net GND: track 298.8 -> 297.8 mm
Other:
- outline, holes or cut-outs redrawn
Changed lines of the file:
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@@
   (general
     (thickness 1.6)
-    (drawings 4)
+    (drawings 8)
     (tracks 623)
     (zones 0)
-    (modules 44)
+    (modules 48)
     (nets 42)
   )
@@
     (uvia_drill 0.1)
   )
+  (module footprint-lib:MountingHole_2.7mm_M2.5,rpi_like locked (layer F.Cu)
+    (at 115 25)
+    (descr "Mounting Hole 2.7mm, no annular, M2.5")
+    (tags "mounting hole 2.7mm no annular m2.5")
+    (attr virtual)
+    (fp_text reference H4 (at 0 -3.7) (layer F.SilkS) hide
+      (effects (font (size 1 1) (thickness 0.15)))
+    )
+    (fp_text value MOUNT_M2.5 (at 0 3.7) (layer F.Fab)
+      (effects (font (size 1 1) (thickness 0.15)))
+    )
+    (fp_circle (center 0 0) (end 1.905 0) (layer B.Mask) (width 1.2))
+    (fp_circle (center 0 0) (end 1.905 0) (layer F.Mask) (width 1.2))
+    (fp_circle (center 0 0) (end 2.95 0) (layer F.CrtYd) (width 0.05))
+    (fp_circle (center 0 0) (end 2.7 0) (layer Cmts.User) (width 0.15))
+    (fp_text user %R (at 0.3 0) (layer F.Fab)
+      (effects (font (size 1 1) (thickness 0.15)))
+    )
+    (pad "" np_thru_hole circle (at 0 0) (size 2.7 2.7) (drill 2.7) (layers *.Cu *.Mask)
+      (solder_mask_margin 1.5) (clearance 1.5))
+  )
+  (module footprint-lib:MountingHole_2.7mm_M2.5,rpi_like locked (layer F.Cu)
+    (at 115 115)
+    (descr "Mounting Hole 2.7mm, no annular, M2.5")
+    (tags "mounting hole 2.7mm no annular m2.5")
+    (attr virtual)
+    (fp_text reference H3 (at 0 -3.7) (layer F.SilkS) hide
+      (effects (font (size 1 1) (thickness 0.15)))
+    )
+    (fp_text value MOUNT_M2.5 (at 0 3.7) (layer F.Fab)
+      (effects (font (size 1 1) (thickness 0.15)))
+    )
+    (fp_circle (center 0 0) (end 1.905 0) (layer B.Mask) (width 1.2))
+    (fp_circle (center 0 0) (end 1.905 0) (layer F.Mask) (width 1.2))
+    (fp_circle (center 0 0) (end 2.95 0) (layer F.CrtYd) (width 0.05))
+    (fp_circle (center 0 0) (end 2.7 0) (layer Cmts.User) (width 0.15))
+    (fp_text user %R (at 0.3 0) (layer F.Fab)
+      (effects (font (size 1 1) (thickness 0.15)))
+    )
+    (pad "" np_thru_hole circle (at 0 0) (size 2.7 2.7) (drill 2.7) (layers *.Cu *.Mask)
+      (solder_mask_margin 1.5) (clearance 1.5))
+  )
+  (module footprint-lib:MountingHole_2.7mm_M2.5,rpi_like locked (layer F.Cu)
+    (at 25 115)
+    (descr "Mounting Hole 2.7mm, no annular, M2.5")
+    (tags "mounting hole 2.7mm no annular m2.5")
+    (attr virtual)
+    (fp_text reference H2 (at 0 -3.7) (layer F.SilkS) hide
+      (effects (font (size 1 1) (thickness 0.15)))
+    )
+    (fp_text value MOUNT_M2.5 (at 0 3.7) (layer F.Fab)
+      (effects (font (size 1 1) (thickness 0.15)))
+    )
+    (fp_circle (center 0 0) (end 1.905 0) (layer B.Mask) (width 1.2))
+    (fp_circle (center 0 0) (end 1.905 0) (layer F.Mask) (width 1.2))
+    (fp_circle (center 0 0) (end 2.95 0) (layer F.CrtYd) (width 0.05))
+    (fp_circle (center 0 0) (end 2.7 0) (layer Cmts.User) (width 0.15))
+    (fp_text user %R (at 0.3 0) (layer F.Fab)
+      (effects (font (size 1 1) (thickness 0.15)))
+    )
+    (pad "" np_thru_hole circle (at 0 0) (size 2.7 2.7) (drill 2.7) (layers *.Cu *.Mask)
+      (solder_mask_margin 1.5) (clearance 1.5))
+  )
+  (module footprint-lib:MountingHole_2.7mm_M2.5,rpi_like locked (layer F.Cu)
+    (at 25 25)
+    (descr "Mounting Hole 2.7mm, no annular, M2.5")
+    (tags "mounting hole 2.7mm no annular m2.5")
+    (attr virtual)
+    (fp_text reference H1 (at 0 -3.7) (layer F.SilkS) hide
+      (effects (font (size 1 1) (thickness 0.15)))
+    )
+    (fp_text value MOUNT_M2.5 (at 0 3.7) (layer F.Fab)
+      (effects (font (size 1 1) (thickness 0.15)))
+    )
+    (fp_circle (center 0 0) (end 1.905 0) (layer B.Mask) (width 1.2))
+    (fp_circle (center 0 0) (end 1.905 0) (layer F.Mask) (width 1.2))
+    (fp_circle (center 0 0) (end 2.95 0) (layer F.CrtYd) (width 0.05))
+    (fp_circle (center 0 0) (end 2.7 0) (layer Cmts.User) (width 0.15))
+    (fp_text user %R (at 0.3 0) (layer F.Fab)
+      (effects (font (size 1 1) (thickness 0.15)))
+    )
+    (pad "" np_thru_hole circle (at 0 0) (size 2.7 2.7) (drill 2.7) (layers *.Cu *.Mask)
+      (solder_mask_margin 1.5) (clearance 1.5))
+  )
   (module footprint-lib:SHT3x-DIS (layer F.Cu)
     (at 107.428499 60.827501 270)
@@
   )
   (module Connector_Pin:Pin_D1.0mm_L10.0mm (layer F.Cu)
-    (at 26.67 25.4)
+    (at 29.5 33.5)
     (descr "solder Pin_ diameter 1.0mm, hole diameter 1.0mm (press fit), length 10.0mm")
     (tags "solder Pin_ press fit")
@@
     )
   )
-  (gr_line (start 120 20) (end 20 20) (layer Edge.Cuts) (width 0.05))
-  (gr_line (start 120 120) (end 120 20) (layer Edge.Cuts) (width 0.05))
-  (gr_line (start 20 120) (end 120 120) (layer Edge.Cuts) (width 0.05))
-  (gr_line (start 20 20) (end 20 120) (layer Edge.Cuts) (width 0.05))
+  (gr_arc (start 115 115) (end 115 120) (angle -90) (layer Edge.Cuts) (width 0.05))
+  (gr_arc (start 25 115) (end 20 115) (angle -90) (layer Edge.Cuts) (width 0.05))
+  (gr_arc (start 25 25) (end 25 20) (angle -90) (layer Edge.Cuts) (width 0.05))
+  (gr_arc (start 115 25) (end 120 25) (angle -90) (layer Edge.Cuts) (width 0.05))
+  (gr_line (start 115 20) (end 25 20) (layer Edge.Cuts) (width 0.05))
+  (gr_line (start 120 115) (end 120 25) (layer Edge.Cuts) (width 0.05))
+  (gr_line (start 25 120) (end 115 120) (layer Edge.Cuts) (width 0.05))
+  (gr_line (start 20 25) (end 20 115) (layer Edge.Cuts) (width 0.05))
   (segment (start 78.458 30.617) (end 78.458 30.617) (width 0.25) (layer B.Cu) (net 1))
   (via (at 74.208 30.512) (size 0.8) (drill 0.4) (layers F.Cu B.Cu) (net 1))
@@
   (segment (start 110.744 55.498999) (end 110.744 56.769) (width 0.25) (layer B.Cu) (net 1))
   (segment (start 108.642 61.306) (end 108.641999 61.556) (width 0.25) (layer B.Cu) (net 1))
-  (segment (start 45.4158 29.2621) (end 45.4158 28.212) (width 0.25) (layer F.Cu) (net 1))
-  (segment (start 39.751 31.369) (end 41.402 29.718) (width 0.25) (layer F.Cu) (net 1))
-  (segment (start 34.085 31.369) (end 39.751 31.369) (width 0.25) (layer F.Cu) (net 1))
-  (segment (start 41.402 29.718) (end 44.9599 29.718) (width 0.25) (layer F.Cu) (net 1))
-  (segment (start 44.9599 29.718) (end 45.4158 29.2621) (width 0.25) (layer F.Cu) (net 1))
   (segment (start 77.2795 39.624004) (end 77.2795 42.9895) (width 0.25) (layer B.Cu) (net 1))
   (segment (start 78.00975 43.71975) (end 79.97825 43.71975) (width 0.25) (layer B.Cu) (net 1))
@@
   (segment (start 112.014001 56.769) (end 110.49 58.293) (width 0.25) (layer B.Cu) (net 2))
   (segment (start 110.49 58.293) (end 110.49 61.356) (width 0.25) (layer B.Cu) (net 2))
-  (segment (start 30.344 30.4115) (end 31.0515 29.704) (width 0.25) (layer F.Cu) (net 2))
   (segment (start 110.236 63.363999) (end 112.2095 63.364) (width 0.25) (layer F.Cu) (net 2))
   (via (at 78.232 37.592) (size 0.8) (drill 0.4) (layers F.Cu B.Cu) (net 2))
@@
   (via (at 55.039464 32.259476) (size 0.8) (drill 0.4) (layers F.Cu B.Cu) (net 24))
   (segment (start 30.9158 24.369) (end 30.9158 24.369) (width 0.25) (layer B.Cu) (net 24))
-  (segment (start 27.701 24.369) (end 26.67 25.4) (width 0.25) (layer B.Cu) (net 24))
-  (segment (start 30.9158 24.369) (end 27.701 24.369) (width 0.25) (layer B.Cu) (net 24))
   (via (at 30.9158 24.369) (size 0.8) (drill 0.4) (layers F.Cu B.Cu) (net 24))
   (segment (start 56.008 23.9545) (end 56.008 26.669) (width 0.25) (layer F.Cu) (net 24))
   (segment (start 56.008 26.669) (end 54.864 27.813) (width 0.25) (layer F.Cu) (net 24))
   (segment (start 54.402988 31.623) (end 55.039464 32.259476) (width 0.25) (layer B.Cu) (net 24))
-  (segment (start 30.861 31.623) (end 54.402988 31.623) (width 0.25) (layer B.Cu) (net 24))
-  (segment (start 29.5038 30.2658) (end 30.861 31.623) (width 0.25) (layer B.Cu) (net 24))
-  (segment (start 29.5038 25.781) (end 29.5038 30.2658) (width 0.25) (layer B.Cu) (net 24))
   (segment (start 30.9158 24.369) (end 29.5038 25.781) (width 0.25) (layer B.Cu) (net 24))
   (segment (start 55.039464 30.528464) (end 55.039464 32.259476) (width 0.25) (layer F.Cu) (net 24))
   (segment (start 54.864 30.353) (end 55.039464 30.528464) (width 0.25) (layer F.Cu) (net 24))
   (segment (start 54.864 27.813) (end 54.864 30.353) (width 0.25) (layer F.Cu) (net 24))
+  (segment (start 33.127 31.623) (end 54.402988 31.623) (width 0.25) (layer B.Cu) (net 24))
+  (segment (start 29.5038 25.781) (end 29.5038 28.7538) (width 0.25) (layer B.Cu) (net 24))
+  (segment (start 29.5 28.7576) (end 29.5 33.5) (width 0.25) (layer B.Cu) (net 24))
+  (segment (start 29.5038 28.7538) (end 29.5 28.7576) (width 0.25) (layer B.Cu) (net 24))
+  (segment (start 31.877 31.623) (end 33.127 31.623) (width 0.25) (layer B.Cu) (net 24))
+  (segment (start 29.623 31.623) (end 31.877 31.623) (width 0.25) (layer B.Cu) (net 24))
+  (segment (start 29.5038 28.7538) (end 29.5038 31.5038) (width 0.25) (layer B.Cu) (net 24))
+  (segment (start 29.5038 31.5038) (end 29.623 31.623) (width 0.25) (layer B.Cu) (net 24))
+  (segment (start 29.5 31.75) (end 29.5 33.5) (width 0.25) (layer B.Cu) (net 24))
+  (segment (start 31.877 31.623) (end 29.627 31.623) (width 0.25) (layer B.Cu) (net 24))
+  (segment (start 29.627 31.623) (end 29.5 31.75) (width 0.25) (layer B.Cu) (net 24))
   (segment (start 61.207072 34.117928) (end 60.708 34.617) (width 0.25) (layer F.Cu) (net 25))
   (segment (start 61.50801 31.69199) (end 61.50801 33.81699) (width 0.25) (layer F.Cu) (net 25))

Commit message: update,
Routing:
- net /MISO: track 34.1 -> 38.4 mm
- net /MOSI: track 40.2 -> 44.5 mm
- net /SCK: track 40.8 -> 37.3 mm
