File: hardware/ESP32-WROOM_tryout.kicad_pcb (KiCad board)
At the start: 2 copper layers, 100 x 100 mm, 48 parts, among them J1 ANT, J2 HEADER1, J3 HEADER2, J4 ANT, J5 I2C_HEADER, J6 SHT3x_HEADER, Q1 2N3904(1AM), Q2 2N3904(1AM), SW1 SW_RESET,2_leg,SMD, SW2 SW_RESET,2_leg,SMD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

Commit message: update,
Routing:
- net /MOSI: track 44.5 -> 34.3 mm
- net /MISO: track 38.4 -> 32.5 mm
- net /SCK: track 37.3 -> 41.8 mm
- net /IO27: track 12.7 -> 15.3 mm
- net /IO25: track 14.4 -> 15.8 mm
Changed lines of the file:
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@@
     (thickness 1.6)
     (drawings 8)
-    (tracks 626)
+    (tracks 625)
     (zones 0)
     (modules 48)
@@
   (segment (start 83.231726 62.995726) (end 86.53 66.294) (width 0.25) (layer B.Cu) (net 8))
   (via (at 74.208 40.672) (size 0.8) (drill 0.4) (layers F.Cu B.Cu) (net 9))
-  (segment (start 65.527581 47.371) (end 64.3255 47.371) (width 0.25) (layer B.Cu) (net 9))
-  (segment (start 67.509 47.371) (end 65.527581 47.371) (width 0.25) (layer B.Cu) (net 9))
-  (segment (start 74.208 40.672) (end 71.215 40.672) (width 0.25) (layer B.Cu) (net 9))
-  (segment (start 69.4415 42.4455) (end 69.4415 45.4385) (width 0.25) (layer B.Cu) (net 9))
-  (segment (start 71.215 40.672) (end 69.4415 42.4455) (width 0.25) (layer B.Cu) (net 9))
-  (segment (start 69.4415 45.4385) (end 67.509 47.371) (width 0.25) (layer B.Cu) (net 9))
+  (segment (start 64.3255 47.371) (end 70.129 47.371) (width 0.25) (layer B.Cu) (net 9))
+  (segment (start 70.129 47.371) (end 70.75 46.75) (width 0.25) (layer B.Cu) (net 9))
+  (segment (start 70.75 41.344) (end 71.422 40.672) (width 0.25) (layer B.Cu) (net 9))
+  (segment (start 70.75 46.75) (end 70.75 41.344) (width 0.25) (layer B.Cu) (net 9))
+  (segment (start 74.208 40.672) (end 71.422 40.672) (width 0.25) (layer B.Cu) (net 9))
   (via (at 74.208 43.212) (size 0.8) (drill 0.4) (layers F.Cu B.Cu) (net 10))
   (segment (start 72.30441 43.212) (end 73.108 43.212) (width 0.25) (layer B.Cu) (net 10))
   (segment (start 73.108 43.212) (end 74.208 43.212) (width 0.25) (layer B.Cu) (net 10))
-  (segment (start 65.60541 49.911) (end 72.30441 43.212) (width 0.25) (layer B.Cu) (net 10))
-  (segment (start 64.3255 49.911) (end 65.60541 49.911) (width 0.25) (layer B.Cu) (net 10))
+  (segment (start 64.3255 49.911) (end 70.089 49.911) (width 0.25) (layer B.Cu) (net 10))
+  (segment (start 71.258205 48.741795) (end 71.258205 44.258205) (width 0.25) (layer B.Cu) (net 10))
+  (segment (start 70.089 49.911) (end 71.258205 48.741795) (width 0.25) (layer B.Cu) (net 10))
+  (segment (start 71.258205 44.258205) (end 72.30441 43.212) (width 0.25) (layer B.Cu) (net 10))
   (via (at 74.208 44.482) (size 0.8) (drill 0.4) (layers F.Cu B.Cu) (net 11))
-  (segment (start 64.3255 52.451) (end 72.2945 44.482) (width 0.25) (layer B.Cu) (net 11))
   (segment (start 72.2945 44.482) (end 73.108 44.482) (width 0.25) (layer B.Cu) (net 11))
   (segment (start 73.108 44.482) (end 74.208 44.482) (width 0.25) (layer B.Cu) (net 11))
@@
   (segment (start 76.1271 65.6271) (end 76 65.5) (width 0.25) (layer F.Cu) (net 11))
   (segment (start 76.1271 69.5744) (end 76.1271 65.6271) (width 0.25) (layer F.Cu) (net 11))
-  (segment (start 72.0725 60.198) (end 75.062815 60.198) (width 0.25) (layer F.Cu) (net 11))
-  (segment (start 75.062815 60.198) (end 75.6285 60.198) (width 0.25) (layer F.Cu) (net 11))
-  (segment (start 64.3255 52.451) (end 72.0725 60.198) (width 0.25) (layer F.Cu) (net 11))
+  (segment (start 75.6285 57.6285) (end 75.6285 60.198) (width 0.25) (layer F.Cu) (net 11))
+  (segment (start 74.5 56.5) (end 75.6285 57.6285) (width 0.25) (layer F.Cu) (net 11))
+  (segment (start 64.3255 52.451) (end 68.3745 56.5) (width 0.25) (layer F.Cu) (net 11))
+  (segment (start 68.3745 56.5) (end 74.5 56.5) (width 0.25) (layer F.Cu) (net 11))
+  (segment (start 64.3255 52.451) (end 69.549 52.451) (width 0.25) (layer B.Cu) (net 11))
+  (segment (start 71.76325 50.23675) (end 71.76325 45.01325) (width 0.25) (layer B.Cu) (net 11))
+  (segment (start 69.549 52.451) (end 71.76325 50.23675) (width 0.25) (layer B.Cu) (net 11))
+  (segment (start 71.76325 45.01325) (end 72.2945 44.482) (width 0.25) (layer B.Cu) (net 11))
   (via (at 74.208 45.752) (size 0.8) (drill 0.4) (layers F.Cu B.Cu) (net 12))
-  (segment (start 73.5645 45.752) (end 74.208 45.752) (width 0.25) (layer B.Cu) (net 12))
-  (via (at 72.1271 65.1229) (size 0.8) (drill 0.4) (layers F.Cu B.Cu) (net 12))
-  (segment (start 72.1271 69.5744) (end 72.1271 65.1229) (width 0.25) (layer F.Cu) (net 12))
-  (segment (start 64.3255 54.991) (end 65.741 54.991) (width 0.25) (layer B.Cu) (net 12))
-  (segment (start 65.741 53.5755) (end 65.78325 53.53325) (width 0.25) (layer B.Cu) (net 12))
-  (segment (start 65.741 54.991) (end 65.741 53.5755) (width 0.25) (layer B.Cu) (net 12))
-  (segment (start 65.78325 53.53325) (end 73.5645 45.752) (width 0.25) (layer B.Cu) (net 12))
-  (segment (start 69.274999 67.975001) (end 71.727101 65.522899) (width 0.25) (layer B.Cu) (net 12))
-  (segment (start 66 55.25) (end 66 66.323002) (width 0.25) (layer B.Cu) (net 12))
-  (segment (start 67.651999 67.975001) (end 69.274999 67.975001) (width 0.25) (layer B.Cu) (net 12))
-  (segment (start 71.727101 65.522899) (end 72.1271 65.1229) (width 0.25) (layer B.Cu) (net 12))
-  (segment (start 65.741 54.991) (end 66 55.25) (width 0.25) (layer B.Cu) (net 12))
-  (segment (start 66 66.323002) (end 67.651999 67.975001) (width 0.25) (layer B.Cu) (net 12))
-  (via (at 74.1271 66) (size 0.8) (drill 0.4) (layers F.Cu B.Cu) (net 13))
-  (segment (start 74.1271 67.8244) (end 74.1271 66) (width 0.25) (layer F.Cu) (net 13))
-  (segment (start 74.1271 69.5744) (end 74.1271 67.8244) (width 0.25) (layer F.Cu) (net 13))
-  (via (at 67 57.5) (size 0.8) (drill 0.4) (layers F.Cu B.Cu) (net 13))
-  (segment (start 64.3255 57.531) (end 64.3255 65.284913) (width 0.25) (layer B.Cu) (net 13))
-  (segment (start 71.702088 68.425012) (end 73.727101 66.399999) (width 0.25) (layer B.Cu) (net 13))
-  (segment (start 64.3255 65.284913) (end 67.465599 68.425012) (width 0.25) (layer B.Cu) (net 13))
-  (segment (start 67.465599 68.425012) (end 71.702088 68.425012) (width 0.25) (layer B.Cu) (net 13))
-  (segment (start 73.727101 66.399999) (end 74.1271 66) (width 0.25) (layer B.Cu) (net 13))
-  (segment (start 64.3255 57.531) (end 66.969 57.531) (width 0.25) (layer F.Cu) (net 13))
-  (segment (start 66.969 57.531) (end 67 57.5) (width 0.25) (layer F.Cu) (net 13))
-  (segment (start 67 57.5) (end 67 53.5) (width 0.25) (layer B.Cu) (net 13))
-  (segment (start 67 53.5) (end 73.258 47.242) (width 0.25) (layer B.Cu) (net 13))
-  (segment (start 73.258 47.242) (end 78.778 47.242) (width 0.25) (layer B.Cu) (net 13))
+  (via (at 72.1271 69.574434) (size 0.8) (drill 0.4) (layers F.Cu B.Cu) (net 12))
+  (segment (start 72.1271 69.5744) (end 72.1271 69.574434) (width 0.25) (layer F.Cu) (net 12))
+  (segment (start 72.1271 69.574434) (end 72.1271 59.3729) (width 0.25) (layer B.Cu) (net 12))
+  (segment (start 71.9952 54.991) (end 72.1271 55.1229) (width 0.25) (layer B.Cu) (net 12))
+  (segment (start 64.3255 54.991) (end 71.9952 54.991) (width 0.25) (layer B.Cu) (net 12))
+  (segment (start 72.1271 59.3729) (end 72.1271 55.1229) (width 0.25) (layer B.Cu) (net 12))
+  (segment (start 74.208 50.292) (end 72.1271 52.3729) (width 0.25) (layer B.Cu) (net 12))
+  (segment (start 74.208 45.752) (end 74.208 50.292) (width 0.25) (layer B.Cu) (net 12))
+  (segment (start 72.1271 55.1229) (end 72.1271 52.3729) (width 0.25) (layer B.Cu) (net 12))
   (segment (start 78.778 47.242) (end 78.778 47.242) (width 0.25) (layer B.Cu) (net 13))
   (via (at 78.778 47.242) (size 0.8) (drill 0.4) (layers F.Cu B.Cu) (net 13))
+  (via (at 74.1271 69.574434) (size 0.8) (drill 0.4) (layers F.Cu B.Cu) (net 13))
+  (segment (start 74.1271 69.5744) (end 74.1271 69.574434) (width 0.25) (layer F.Cu) (net 13))
+  (segment (start 74.1271 69.574434) (end 73 68.447334) (width 0.25) (layer B.Cu) (net 13))
+  (via (at 73 57.5) (size 0.8) (drill 0.4) (layers F.Cu B.Cu) (net 13))
+  (segment (start 73 58.065685) (end 73 57.5) (width 0.25) (layer B.Cu) (net 13))
+  (segment (start 72.969 57.531) (end 73 57.5) (width 0.25) (layer F.Cu) (net 13))
+  (segment (start 73 68.447334) (end 73 58.065685) (width 0.25) (layer B.Cu) (net 13))
+  (segment (start 64.3255 57.531) (end 72.969 57.531) (width 0.25) (layer F.Cu) (net 13))
+  (segment (start 73 52.32) (end 73 56.934315) (width 0.25) (layer B.Cu) (net 13))
+  (segment (start 73 56.934315) (end 73 57.5) (width 0.25) (layer B.Cu) (net 13))
+  (segment (start 78.078 47.242) (end 73 52.32) (width 0.25) (layer B.Cu) (net 13))
+  (segment (start 78.778 47.242) (end 78.078 47.242) (width 0.25) (layer B.Cu) (net 13))
   (via (at 52.9844 29.464) (size 0.8) (drill 0.4) (layers F.Cu B.Cu) (net 14))
   (segment (start 51.558 29.582) (end 52.8664 29.582) (width 0.25) (layer F.Cu) (net 14))
