File: hardware/ESP32-WROOM_tryout.kicad_pcb (KiCad board)
At the start: 2 copper layers, 100 x 100 mm, 48 parts, among them J1 ANT, J2 HEADER1, J3 HEADER2, J4 ANT, J5 I2C_HEADER, J6 SHT3x_HEADER, Q1 2N3904(1AM), Q2 2N3904(1AM), SW1 SW_RESET,2_leg,SMD, SW2 SW_RESET,2_leg,SMD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

Commit message: in the middle,
Parts:
- added C1: C106,0805, Capacitor_SMD:C_0805_2012Metric_Pad1.15x1.40mm_HandSolder, F.Cu at (42.0, 108.5)
- added D1: D_1N4148_T4, Diode_SMD:D_SOD-123, F.Cu at (33.1, 105.3)
- added D2: D_1N4148_T4, Diode_SMD:D_SOD-123, F.Cu at (33.1, 107.8)
- added D3: LED_ORANGE,0603, footprint-lib:LED_0603_1608Metric, F.Cu at (48.6, 108.0)
- added D4: LED_GREEN,0603, footprint-lib:LED_0603_1608Metric, F.Cu at (46.7, 108.0)
- added D5: LED_RED,0603, footprint-lib:LED_0603_1608Metric, F.Cu at (44.9, 107.9)
- added F1: Fuse_Small,0805, Resistor_SMD:R_0805_2012Metric_Pad1.15x1.40mm_HandSolder, F.Cu at (42.7, 112.0)
- added J1: OUT_HEADER, Connector_PinHeader_1.27mm:PinHeader_1x03_P1.27mm_Vertical, F.Cu at (26.7, 105.7)
- added R1: R103,0603, Resistor_SMD:R_0603_1608Metric_Pad1.05x0.95mm_HandSolder, F.Cu at (38.2, 111.0)
- added R2: R122,0603, Resistor_SMD:R_0603_1608Metric_Pad1.05x0.95mm_HandSolder, B.Cu at (48.6, 108.0)
- added R3: R122,0603, Resistor_SMD:R_0603_1608Metric_Pad1.05x0.95mm_HandSolder, B.Cu at (46.7, 108.0)
- added R4: R122,0603, Resistor_SMD:R_0603_1608Metric_Pad1.05x0.95mm_HandSolder, F.Cu at (40.0, 111.0)
- added R5: R122,0603, Resistor_SMD:R_0603_1608Metric_Pad1.05x0.95mm_HandSolder, B.Cu at (44.9, 108.0)
- added U1: USB_Micro, footprint-lib:USB_Micro-B_Molex-105017-0001, F.Cu at (36.5, 117.3)
- added U2: MCP73837_MSOP10, footprint-lib:MCP73837_MSOP10, F.Cu at (33.1, 110.9)
Routing:
- net GND: track 298.2 -> 350.6 mm, vias 11 -> 15
- net Net-(R2-Pad1): track 0.00 -> 27.8 mm, vias 0 -> 1
- net +5V: track 51.3 -> 74.7 mm, vias 2 -> 3
- net Net-(R3-Pad1): track 0.00 -> 23.2 mm, vias 0 -> 1
- net Net-(D1-Pad1): track 1.80 -> 22.6 mm
- net Vout: track 0.00 -> 20.5 mm, vias 0 -> 1
- net Net-(R5-Pad1): track 0.00 -> 12.6 mm, vias 0 -> 1
- net Net-(F1-Pad1): track 0.00 -> 9.45 mm, vias 0 -> 2
- net Net-(R4-Pad2): track 0.00 -> 6.75 mm
- net Net-(R1-Pad2): track 0.00 -> 3.78 mm
- net Net-(D2-Pad2): track 2.04 -> 4.29 mm
- net /SCK: track 41.8 -> 43.5 mm
- net Net-(D5-Pad1): vias 0 -> 1
- net Net-(D4-Pad1): vias 0 -> 1
- net Net-(D3-Pad1): vias 0 -> 1
Other:
- net class 800mA removed
- net class GND removed
- board text added: "ESP32-WROOM_tryout"
- board text added: "MCP73837-tryout"
- board text added: "SHT30_tryout"
- board text added: "git@github.com:louiscklaw/ESP32-WROOM_tryout.git git@github.com:louiscklaw/SHT30_tryout.git git@github.com:louiscklaw/MCP73837-tryout.git"

Commit message: update,
Parts:
- added J7: TTL_DEBUG, Connector_PinHeader_2.54mm:PinHeader_1x03_P2.54mm_Vertical, F.Cu at (63.2, 23.2)
Connections:
- RN1 pad 3: (no net) -> Net-(RN1-Pad3)
- RN1 pad 4: (no net) -> Net-(RN1-Pad4)
- U1 pad 17: (no net) -> Net-(U1-Pad17)
- U1 pad 18: (no net) -> Net-(U1-Pad18)
- U1 pad 19: (no net) -> Net-(U1-Pad19)
- U1 pad 20: (no net) -> Net-(U1-Pad20)
- U1 pad 21: (no net) -> Net-(U1-Pad21)
- U1 pad 22: (no net) -> Net-(U1-Pad22)
- U1 pad 23: (no net) -> Net-(U1-Pad23)
- U1 pad 24: (no net) -> Net-(U1-Pad24)
- U1 pad 32: (no net) -> Net-(U1-Pad32)
- U1 pad 4: (no net) -> Net-(U1-Pad4)
- U1 pad 5: (no net) -> Net-(U1-Pad5)
- U1 pad 6: (no net) -> Net-(U1-Pad6)
- U1 pad 7: (no net) -> Net-(U1-Pad7)
- U2 pad 11: (no net) -> Net-(U2-Pad11)
- U2 pad 12: (no net) -> Net-(U2-Pad12)
- U2 pad 7: (no net) -> Net-(U2-Pad7)
- U3 pad 4: (no net) -> Net-(U3-Pad4)
- U4 pad 10: (no net) -> Net-(U4-Pad10)
- U4 pad 11: (no net) -> Net-(U4-Pad11)
- U4 pad 12: (no net) -> Net-(U4-Pad12)
- U4 pad 15: (no net) -> Net-(U4-Pad15)
- U4 pad 7: (no net) -> Net-(U4-Pad7)
- U4 pad 8: (no net) -> Net-(U4-Pad8)
- U4 pad 9: (no net) -> Net-(U4-Pad9)
Routing:
- net /RXI: track 67.1 -> 73.5 mm, vias 3 -> 4
- net GND: track 350.6 -> 356.9 mm
- net /TXO: track 70.2 -> 75.6 mm, vias 3 -> 4
